File: PCB/Revolve_A0/Revolve_A0.sch (EAGLE design)
At the start: 441 parts, among them IC1 TMC2100-LA, IC10 74AHC1G126DCK, IC11 74AHC1G126DCK, IC12 TMC2100-LA, IC13 74AHC1G126DCK, IC14 74AHC1G126DCK, IC15 TMC2100-LA, IC16 74AHC1G126DCK, IC17 74AHC1G126DCK, IC18 74AHC1G126DCK, IC19 74AHC1G126DCK, IC2 TMC2100-LA, IC20 74AHC1G126DCK, IC21 74AHC1G126DCK, IC22 74AHC1G126DCK, IC24 TMC2100-LA, IC25 74AHC1G126DCK, IC26 74AHC1G126DCK, IC27 74AHC1G126DCK, IC28 74AHC1G126DCK, IC29 LAN8710A, IC3 74AHC1G126DCK, IC30 MTFC2GMDEA, IC31 CY7C65632, IC4 74AHC1G126DCK, IC5 TMC2100-LA, IC6 74AHC1G126DCK, IC7 74AHC1G126DCK, IC8 74AHC1G126DCK, IC9 74AHC1G126DCK, J1 USD_CONNECTOR, Q1 AON6758, Q2 AON6758, Q3 AON6758, Q8 AON6758, U1 SN74AHC595PW, U10 TPD4S012_DRY_6, U11 PCA9685PW, U18 CAT24C256, U19 CD4050BD, U2 SN74AHC595PW, U3 SN74AHC595PW, U4 SN74AHC595PW, U5 SN74AHC595PW, U6 RT8268, U8 SN74AHC595PW, X1 22-05-7038-03, X10 22-05-7038-03, X11 22-05-7038-03, X12 22-05-7048-04, X13 22-05-7038-03, X14 22-05-7048-04, X15 22-05-7048-04, X16 22-05-7048-04, X17 22-05-7048-04, X18 22-05-7048-04, X19 22-05-7038-03, X2 MSTBA4, X20 MSTBA4, X21 MSTBA2, X22 22-05-7038-03, X23 22-05-7038-03, X24 HDMI, X25 22-05-7048-04, X26 MSTBA2, X27 MINI-USB_SHIELD5P4-32005-400, X29 22-05-7038-03, X3 MSTBA2, X4 22-05-7028-02, X5 22-05-7028-02, X6 22-05-7028-02, X7 22-05-7038-03, X8 22-05-7038-03, X9 22-05-7028-02, Y1 24MHz, Y2 32.768 MHz, Y3 25 MHz, Y4 12 MHz

Commit message: Starting up work again
Parts:
- removed C14, C15, C24, C41, C42, C5, C84, C85, C86, C87, C88, C99: 0.1uF, rcl:C-EUC0402
- removed IC10, IC11, IC13, IC14, IC16, IC17, IC18, IC19, IC20, IC21, IC22, IC25, IC26, IC27, IC3, IC4, IC8, IC9: 74AHC1G126DCK, 74xx-little-de:74AHC1G126DCK
- removed U1, U2, U3, U4, U5, U8: SN74AHC595PW, sn74hc595:SN74AHC595PW
Connections:
- removed net EN_EHA: IC19A.I, IC22A.I, IC27A.I, U4.QA
- removed net EN_XYZ: IC18A.I, IC20A.I, IC21A.I, U1.QA
- removed net N$103: IC17A.OE, U5.QH
- removed net N$104: IC17A.I, U5.QG
- removed net N$105: IC16A.OE, U5.QF
- removed net N$106: IC16A.I, U5.QE
- removed net N$142: IC26A.OE, U8.QH
- removed net N$143: IC26A.I, U8.QG
- removed net N$144: IC25A.I, U8.QE
- removed net N$146: IC25A.OE, U8.QF
- removed net N$34: IC3A.I, U1.QE
- removed net N$4: IC4A.OE, U1.QH
- removed net N$40: IC3A.OE, U1.QF
- removed net N$5: IC4A.I, U1.QG
- removed net N$59: IC11A.OE, U3.QH
- removed net N$61: IC11A.I, U3.QG
- removed net N$62: IC10A.OE, U3.QF
- removed net N$63: IC10A.I, U3.QE
- removed net N$66: IC9A.OE, U2.QH
- removed net N$67: IC9A.I, U2.QG
- removed net N$68: IC8A.OE, U2.QF
- removed net N$69: IC8A.I, U2.QE
- removed net N$85: IC14A.OE, U4.QH
- removed net N$86: IC14A.I, U4.QG
- removed net N$87: IC13A.OE, U4.QF
- removed net N$93: IC13A.I, U4.QE
- removed net SER6: U5.QH_2
- removed net SER_2: U1.QH_2, U2.SER
- removed net SER_3: U2.QH_2, U3.SER
- removed net SER_4: U3.QH_2, U4.SER
- removed net SER_5: U4.QH_2, U5.SER
- removed net SER_6: U8.SER
- removed net TRISTATE_STEPPERS: IC18A.OE, IC19A.OE, IC20A.OE, IC21A.OE, IC22A.OE, IC27A.OE, U5.QA, U8.QA
- net +3V3: no longer C14.1, C15.1, C24.1, C41.1, C42.1, C5.1, C84.1, C85.1, C86.1, C87.1, C88.1, C99.1, IC10P.VCC, IC11P.VCC, IC13P.VCC, IC14P.VCC, IC16P.VCC, IC17P.VCC, IC18P.VCC, IC19P.VCC, IC20P.VCC, IC21P.VCC, IC22P.VCC, IC25P.VCC, IC26P.VCC, IC27P.VCC, IC3P.VCC, IC4P.VCC, IC8P.VCC, IC9P.VCC, U1.VCC, U1.~SRCLR, U2.VCC, U2.~SRCLR, U3.VCC, U3.~SRCLR, U4.VCC, U4.~SRCLR, U5.VCC, U5.~SRCLR, U8.VCC, U8.~SRCLR
- net ENABLE_A: no longer IC27A.O
- net ENABLE_E: no longer IC19A.O
- net ENABLE_H: no longer IC22A.O
- net ENABLE_X: no longer IC18A.O
- net ENABLE_Y: no longer IC20A.O
- net ENABLE_Z: no longer IC21A.O
- net GND: no longer C14.2, C15.2, C24.2, C41.2, C42.2, C5.2, C84.2, C85.2, C86.2, C87.2, C88.2, C99.2, IC10P.GND, IC11P.GND, IC13P.GND, IC14P.GND, IC16P.GND, IC17P.GND, IC18P.GND, IC19P.GND, IC20P.GND, IC21P.GND, IC22P.GND, IC25P.GND, IC26P.GND, IC27P.GND, IC3P.GND, IC4P.GND, IC8P.GND, IC9P.GND, U1.GND, U1.~OE, U2.GND, U2.~OE, U3.GND, U3.~OE, U4.GND, U4.~OE, U5.GND, U5.~OE, U8.GND, U8.~OE
- net N$100: no longer U5.QD
- net N$101: no longer U5.QC
- net N$102: no longer U5.QB
- net N$133: no longer IC25A.O
- net N$138: no longer IC26A.O
- net N$139: no longer U8.QD
- net N$140: no longer U8.QC
- net N$141: no longer U8.QB
- net N$28: no longer IC10A.O
- net N$42: no longer IC8A.O
- net N$43: no longer U1.QB
- net N$44: no longer U1.QD
- net N$49: no longer IC9A.O
- net N$53: no longer U2.QD
- net N$54: no longer IC11A.O
- net N$55: no longer U3.QD
- net N$56: no longer U2.QC
- net N$57: no longer U3.QC
- net N$58: no longer U3.QB
- net N$6: no longer U1.QC
- net N$65: no longer U2.QB
- net N$76: no longer IC13A.O
- net N$81: no longer IC14A.O
- net N$82: no longer U4.QD
- net N$83: no longer U4.QC
- net N$84: no longer U4.QB
- net N$91: no longer IC16A.O
- net N$99: no longer IC17A.O
- net SERVO_0_EN: no longer U2.QA
- net SERVO_1_EN: no longer U3.QA
- net SPI1_CS1: no longer U1.RCLK, U2.RCLK, U3.RCLK, U4.RCLK, U5.RCLK, U8.RCLK
- net SPI1_MOSI: no longer U1.SER
- net SPI1_SCLK: no longer U1.SRCLK, U2.SRCLK, U3.SRCLK, U4.SRCLK, U5.SRCLK, U8.SRCLK
- net X_CFG1: no longer IC4A.O
- net X_CFG2: no longer IC3A.O

Commit message: Started porting to SIP-SM, changed to TMC2130
Parts:
- removed C13, C153: 0.1uF, rcl:C-EUC0402
- removed C154: 10uF, rcl:C-EUC0402
- removed IC28: 74AHC1G126DCK, 74xx-little-de:74AHC1G126DCK
- removed J1: USD_CONNECTOR, BeagleBone_Blue:USD_CONNECTOR
- removed R142, R143, R144, R145, R146: 4.7K, rcl:R-EU_R0402
- removed TP1, TP2, TP3, TP4: TPPAD1-13, testpad:TPPAD1-13
- removed U$10, U$8: IP4283CZ10-TBR, Revolve:IP4283CZ10-TBR
- removed U18: CAT24C256, custom:CAT24C256
- removed Y2: 32.768 MHz, Revolve:445C33D24M000003.2X1.5
- added C15, C24, C84, C85, C87, C99: 0.1uF, rcl:C-EUC0402
- added C41: 10uF, rcl:C-EUC0805
- added C42: 100uF, Panasonic-EEEFK_EEEFP:C
- added C86: 4.7uF, rcl:C-EUC0402
- added C88: 22nF, rcl:C-EUC0402
- added EEPROM_WP, PMIC_NRESET, SYS_5V, SYS_RTC_1V8, SYS_VDD1_3V3, SYS_VDD2_3V3, SYS_VDD3_3V3, VDDS_DDR, VDDS_PLL, VDD_CODE, VDD_MPU: TPPAD1-13, testpad:TPPAD1-13
- added R153: 22R, rcl:R-EU_R0402
- added SV2: (no value), con-lstb:MA05-1
- added U$11, U$12: DF10G7M1N, Revolve:DF10G7M1N
- added U1: OSD3358-512M-BSM, Octavo-Systems:OSD3358-512M-BSM
- C144, C145: value 18pF -> 4.7uF
- C152: value 0.1uF -> 0.001uF
- R126: value 22R -> 2.2R; MPN RC0402JR-074K7L -> RC1005J2R2CS
- R138: value 4.7K -> 0.1R; device rcl:R-EU_R0402 -> rcl:R-EU_R0805; MPN RC0402JR-074K7L -> RL1220S-R10-F
- R139: value 1.5K -> 0.1R; device rcl:R-EU_R0402 -> rcl:R-EU_R0805; MPN RC0402JR-074K7L -> RL1220S-R10-F
- R140: value 1.5K -> 10K; MPN RC0402JR-074K7L -> RC0402FR-0710KL
- R141: value 4.7K -> 10K; MPN RC0402JR-074K7L -> RC0402FR-0710KL
- R149: value 1M -> 0.1,5%; MPN RC0402JR-074K7L -> RC1005F4422CS
- U$2: value OSD3358-PARTS -> TRINAMIC_TMC2130_QFN36; device OSD3358-BAS-2:OSD3358-PARTS -> TMC2130-Eval_v13:TRINAMIC_TMC2130_QFN36
Connections:
- removed net GPIO1_16: U$2G$1.GPMC_A00
- removed net GPIO2_0: U$2G$1.GPMC_CSN3
- removed net GPIO3_21: U$2G$1.GPMC_A11
- removed net LCD_VCLK: R126.1, U$7.PCLK
- removed net LDO_PGOOD: U$2G$1.RTC_PWRONRSTN, U$2G$3.PMIC_OUT_LDO_PGOOD
- removed net MMC0_CD: J1.CD1, R146.1, U$2G$1.SPI0_CS1
- removed net MMC0_CLK: J1.CLK, R138.1, U$2G$1.MMC0_CLK
- removed net MMC0_CMD: J1.CMD, R141.1, U$2G$1.MMC0_CMD
- removed net MMC0_DAT0: J1.DAT0, R142.1, U$2G$1.MMC0_DAT0
- removed net MMC0_DAT1: J1.DAT1, R143.1, U$2G$1.MMC0_DAT1
- removed net MMC0_DAT2: J1.DAT2, R144.1, U$2G$1.MMC0_DAT2
- removed net MMC0_DAT3: J1.CD/DAT3, R145.1, U$2G$1.MMC0_DAT3
- removed net N$182: U$2G$1.MCASP0_AXR1
- removed net N$211: U$2G$1.GPMC_ADVN_ALE
- removed net PMIC_INT: U$2G$3.PMIC_OUT_NINT
- removed net PMIC_NWAKEUP: U$2G$1.EXT_WAKEUP, U$2G$3.PMIC_OUT_NWAKEUP
- removed net PMIC_PGOOD: IC28A.I, U$2G$1.PWRONRSTN, U$2G$3.PMIC_OUT_PGOOD
- removed net PMIC_POWER_EN: U$2G$3.PMIC_IN_PWR_EN, U$2G$3.PMIC_POWER_EN
- removed net SPI1_CS1: U$2G$2.ECAP0_IN_PWM0_OUT
- removed net SPI1_MISO: U$2G$2.MCASP0_FSX
- removed net SPI1_MOSI: U$2G$2.MCASP0_AXR0
- removed net SPI1_SCLK: U$2G$2.MCASP0_ACLKX
- removed net VDD_1V8: L3.2, U$2G$3.SYS_VDD_1P8V_N16, U$2G$3.SYS_VDD_1P8V_R16
- removed net VDD_3V3A: U$2G$5.VDDSHV_3P3V_E10, U$2G$5.VDDSHV_3P3V_E11, U$2G$5.VDDSHV_3P3V_E12, U$2G$5.VDDSHV_3P3V_E13, U$2G$5.VDDSHV_3P3V_F14, U$2G$5.VDDSHV_3P3V_G14, U$2G$5.VDDSHV_3P3V_H14, U$2G$5.VDDSHV_3P3V_J14, U$2G$5.VDDSHV_3P3V_K14, U$2G$5.VDDSHV_3P3V_L14, U$2G$5.VDDSHV_3P3V_N15, U$2G$5.VDDSHV_3P3V_N5, U$2G$5.VDDSHV_3P3V_P10, U$2G$5.VDDSHV_3P3V_P11, U$2G$5.VDDSHV_3P3V_P12, U$2G$5.VDDSHV_3P3V_P13, U$2G$5.VDDSHV_3P3V_P5, U$2G$5.VDDSHV_3P3V_P6, U$2G$5.VDDSHV_3P3V_P7, U$2G$5.VDDSHV_3P3V_P8, U$2G$5.VDDSHV_3P3V_R15
- removed net VDD_3V3AUX: R89.2, U$2G$3.SYS_VDD2_3P3V
- removed net VDD_RTC: IC28A.OE, IC28P.VCC, U$2G$5.SYS_RTC_1P8V_D7, U$2G$5.SYS_RTC_1P8V_E14, U$2G$5.SYS_RTC_1P8V_E6, U$2G$5.SYS_RTC_1P8V_F9, U$2G$5.SYS_RTC_1P8V_K13, U$2G$5.SYS_RTC_1P8V_N6, U$2G$5.SYS_RTC_1P8V_P14, U$2G$5.SYS_RTC_1P8V_P9
- new net CGND: R149.2
- new net DIR_B: U1C.MMC0_CLK
- new net DIR_C: U1C.GPMC_AD13
- new net IREF_X1: C145.1, R140.2, R141.1
- new net LCD_PCLK: R153.1, U$7.PCLK, U1D.LCD_PCLK
- new net N$103: U1A.I2C0_SCL, U1A.PMIC_SCL
- new net N$104: U1A.I2C0_SDA, U1A.PMIC_SDA
- new net N$105: SYS_VDD1_3V3.TP, U1A.SYS_VDD1_3P3V@1, U1A.SYS_VDD1_3P3V@2, U1A.SYS_VDD1_3P3V@3, U1A.SYS_VDD1_3P3V@4
- new net N$106: U$2.SWP_DIAG1
- new net N$120: SYS_VDD3_3V3.TP, U1A.SYS_VDD3_3P3V@1, U1A.SYS_VDD3_3P3V@2, U1A.SYS_VDD3_3P3V@3, U1A.SYS_VDD3_3P3V@4, U1A.SYS_VDD3_3P3V@5, U1A.SYS_VDD3_3P3V@6, U1A.SYS_VDD3_3P3V@7, U1A.SYS_VDD3_3P3V@8
- new net N$142: SYS_RTC_1V8.TP, U1A.SYS_RTC_1P8V@1, U1A.SYS_RTC_1P8V@2
- new net N$143: U1A.EXT_WAKEUP, U1A.PMIC_NWAKEUP
- new net N$144: U1A.EXTINTN, U1A.PMIC_NINT
- new net N$146: U1A.VDDSHV1, U1A.VDDSHV2, U1A.VDDSHV3, U1A.VDDSHV4, U1A.VDDSHV5, U1A.VDDSHV6
- new net N$161: U$2.SWN_DIAG0
- new net N$162: PMIC_NRESET.TP, U1A.PMIC_NRESET
- new net N$165: U1C.GPMC_CLK
- new net N$166: C86.2, R126.1, U$2.5VOUT
- new net N$167: C87.1, R126.2, U$2.VCC
- new net N$168: C88.2, U$2.CPO
- new net N$170: C88.1, U$2.CPI
- new net N$171: C99.1, U$2.VCP
- new net N$188: U1C.GPMC_A1
- new net N$189: U1C.GPMC_A2
- new net N$190: U1C.GPMC_A3
- new net N$215: SV2.4, U1C.UART0_RXD
- new net N$34: U1F.VDDS_DDR, VDDS_DDR.TP
- new net N$4: SV2.3, U1C.UART0_CTSN
- new net N$40: U1F.VDD_CORE, VDD_CODE.TP
- new net N$5: SV2.2, U1C.UART0_RTSN
- new net SPI0_CS0: U1C.SPI0_CS0
- new net SPI0_CS1: U1C.SPI0_CS1
- new net SPI0_CSX: U$2.CSN_CFG3
- new net SPI0_MISO: U$2.SDO_NAO_CFG0, U1C.SPI0_D0
- new net SPI0_MOSI: U$2.SDI_NAI_CFG1, U1C.SPI0_D1
- new net SPI0_SCLK: U$2.SCK_CFG2, U1C.SPI0_SCLK
- new net STEP_B: U1C.MMC0_CMD
- new net STEP_C: U1C.GPMC_AD12
- new net SYS_VDD2_3V3: R89.2, SYS_VDD2_3V3.TP, U1A.SYS_VDD2_3P3V@1, U1A.SYS_VDD2_3P3V@2
- new net SYS_VDD_1V8: L3.2, U1A.SYS_VDD_1P8V@1, U1A.SYS_VDD_1P8V@2, U1A.SYS_VDD_1P8V@3, U1A.SYS_VDD_1P8V@4, U1A.SYS_VDD_1P8V@5, U1A.SYS_VDD_1P8V@6, U1A.SYS_VDD_1P8V@7, U1A.SYS_VDD_1P8V@8
- new net VDDS_PLL: U1F.VDDS_PLL, VDDS_PLL.TP
- new net VDD_MPU: U1F.VDD_MPU, VDD_MPU.TP
- net +24V: now also C15.1, C24.1, C41.1, C42.+, C85.2, C99.2, U$2.VS, U$2.VSA
- net +3V3: now also C84.1, U$2.VCC_IO; no longer C13.1, C153.1, C154.1, J1.VCC, R138.2, R139.2, R140.2, R141.2, R142.2, R143.2, R144.2, R145.2, R146.2, U$2G$3.SYS_VDD1_3P3V_U20, U$2G$3.SYS_VDD1_3P3V_V20, U18.A2, U18.VCC
- net +5V: now also U1A.VIN_AC@1, U1A.VIN_AC@2, U1A.VIN_AC@3; no longer U$2G$3.VIN_AC_Y5, U$2G$3.VIN_AC_Y6
- net DIR_A: now also U1C.MMC0_DAT0
- net DIR_E: now also U1C.MCASP0_AHCLKX; no longer U$2G$1.GPMC_AD15
- net DIR_H: now also U1C.MMC0_DAT2; no longer U$2G$1.GPMC_AD14
- net DIR_X: now also U$2.REFR_DIR, U1C.MCASP0_FSX; no longer U$2G$1.GPMC_CSN0
- net DIR_Y: now also U1C.MCASP0_AHCLKR; no longer U$2G$1.GPMC_AD08
- net DIR_Z: now also U1C.MCASP0_FSR; no longer U$2G$1.GPMC_AD10
- net EMMC_RST: now also U1C.GPMC_A4; no longer U$2G$1.GPMC_A04
- net ENABLE: no longer U$2G$1.XDMA_EVENT_INTR1
- net END_STOP_X_1: no longer U$2G$2.MCASP0_AHCLKX
- net END_STOP_X_2: no longer U$2G$1.GPMC_WAIT0
- net END_STOP_Y_1: no longer U$2G$1.GPMC_A01
- net END_STOP_Y_2: no longer U$2G$2.MCASP0_AHCLKR
- net END_STOP_Z_1: no longer U$2G$1.GPMC_WPN
- net END_STOP_Z_2: no longer U$2G$2.SPI0_D1
- net FAULT_E: no longer U$2G$1.GPMC_CLK
- net FAULT_H: no longer U$2G$1.GPMC_OEN_REN
- net FAULT_X: no longer U$2G$1.GPMC_WEN
- net FAULT_Y: no longer U$2G$1.GPMC_BEN0_CLE
- net FAULT_Z: no longer U$2G$2.UART1_TXD
- net GND: now also C144.2, C145.2, C15.2, C24.2, C41.2, C42.-, C84.2, C85.1, C86.1, C87.2, R138.1, R139.1, R149.1, SV2.1, U$11.GND, U$12.GND, U$2.GND, U$2.GNDA, U$2.TST_MODE, U1E.DGND@1, U1E.DGND@10, U1E.DGND@11, U1E.DGND@12, U1E.DGND@13, U1E.DGND@14, U1E.DGND@15, U1E.DGND@16, U1E.DGND@17, U1E.DGND@18, U1E.DGND@19, U1E.DGND@2, U1E.DGND@20, U1E.DGND@21, U1E.DGND@22, U1E.DGND@23, U1E.DGND@24, U1E.DGND@25, U1E.DGND@26, U1E.DGND@27, U1E.DGND@28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; no longer C13.2, C153.2, C154.2, IC28P.GND, J1.GND, J1.SHIELD@1, J1.SHIELD@3, U$10.GND1, U$10.GND2, U$2G$4.VSS_A1, U$2G$4.VSS_A18, U$2G$4.VSS_E19, U$2G$4.VSS_E20, U$2G$4.VSS_F19, U$2G$4.VSS_F8, U$2G$4.VSS_G11, U$2G$4.VSS_G12, U$2G$4.VSS_G19, U$2G$4.VSS_G8, U$2G$4.VSS_G9, U$2G$4.VSS_H10, U$2G$4.VSS_H12, U$2G$4.VSS_H19, U$2G$4.VSS_H6, U$2G$4.VSS_H7, U$2G$4.VSS_H8, U$2G$4.VSS_H9, U$2G$4.VSS_J10, U$2G$4.VSS_J11, U$2G$4.VSS_J19, U$2G$4.VSS_J20, U$2G$4.VSS_J6, U$2G$4.VSS_J7, U$2G$4.VSS_J8, U$2G$4.VSS_J9, U$2G$4.VSS_K10, U$2G$4.VSS_K11, U$2G$4.VSS_K19, U$2G$4.VSS_K7, U$2G$4.VSS_K9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
- net GNDA_ADC: now also U1B.AGND_ADC; no longer U$2G$2.VSSA_ADC_A6, U$2G$2.VSSA_ADC_A9, U$2G$2.VSSA_ADC_E8
- net HDMI_INT: now also U1C.GPMC_A9; no longer U$2G$1.GPMC_A09
- net I2C0_SCL: no longer R140.1, U$2G$3.I2C0_SCL, U$2G$3.PMIC_IN_I2C_SCL, U18.SCL
- net I2C0_SDA: no longer R139.1, U$2G$3.I2C0_SDA, U$2G$3.PMIC_IN_I2C_SDA, U18.SDA
- net IREF_X_RAW: now also R141.2
- net LCD_D0: now also U1D.LCD_DATA0; no longer U$2G$2.LCD_DATA00
- net LCD_D1: now also U1D.LCD_DATA1; no longer U$2G$2.LCD_DATA01
- net LCD_D10: now also U1D.LCD_DATA10; no longer U$2G$2.LCD_DATA10
- net LCD_D11: now also U1D.LCD_DATA11; no longer U$2G$2.LCD_DATA11
- net LCD_D12: now also U1D.LCD_DATA12; no longer U$2G$2.LCD_DATA12
- net LCD_D13: now also U1D.LCD_DATA13; no longer U$2G$2.LCD_DATA13
- net LCD_D14: now also U1D.LCD_DATA14; no longer U$2G$2.LCD_DATA14
- net LCD_D15: now also U1D.LCD_DATA15; no longer U$2G$2.LCD_DATA15
- net LCD_D2: now also U1D.LCD_DATA2; no longer U$2G$2.LCD_DATA02
- net LCD_D3: now also U1D.LCD_DATA3; no longer U$2G$2.LCD_DATA03
- net LCD_D4: now also U1D.LCD_DATA4; no longer U$2G$2.LCD_DATA04
- net LCD_D5: now also U1D.LCD_DATA5; no longer U$2G$2.LCD_DATA05
- net LCD_D6: now also U1D.LCD_DATA6; no longer U$2G$2.LCD_DATA06
- net LCD_D7: now also U1D.LCD_DATA7; no longer U$2G$2.LCD_DATA07
- net LCD_D8: now also U1D.LCD_DATA8; no longer U$2G$2.LCD_DATA08
- net LCD_D9: now also U1D.LCD_DATA9; no longer U$2G$2.LCD_DATA09
- net LCD_DE: now also R153.2, U1D.LCD_AC_BIAS_EN; no longer U$2G$2.LCD_AC_BIAS_EN
- net LCD_HSYNC: now also U1D.LCD_HSYNC; no longer U$2G$2.LCD_HSYNC
- net LCD_VSYNC: now also U1D.LCD_VSYNC; no longer U$2G$2.LCD_VSYNC
- net MDIO_CLK: now also U1D.MDC; no longer U$2G$2.MDC
- net MDIO_DATA: now also U1D.MDIO; no longer U$2G$2.MDIO
- net MII1_COL: now also U1D.MII1_COL; no longer U$2G$2.MII1_COL
- net MII1_CRS_DV: now also U1D.MII1_CRS; no longer U$2G$2.MII1_CRS
- net MII1_RXCLK: now also U1D.MII1_RX_CLK; no longer U$2G$2.MII1_RX_CLK
- net MII1_RXD0: now also U1D.MII1_RXD0; no longer U$2G$2.MII1_RXD0
- net MII1_RXD1: now also U1D.MII1_RXD1; no longer U$2G$2.MII1_RXD1
- net MII1_RXD2: now also U1D.MII1_RXD2; no longer U$2G$2.MII1_RXD2
- net MII1_RXD3: now also U1D.MII1_RXD3; no longer U$2G$2.MII1_RXD3
- net MII1_RXDV: now also U1D.MII1_RX_DV; no longer U$2G$2.MII1_RX_DV
- net MII1_RXERR: now also U1D.MII1_RX_ER; no longer U$2G$2.MII1_RX_ER
- net MII1_TXCLK: now also U1D.MII1_TX_CLK; no longer U$2G$2.MII1_TX_CLK
- net MII1_TXD0: now also U1D.MII1_TXD0; no longer U$2G$2.MII1_TXD0
- net MII1_TXD1: now also U1D.MII1_TXD1; no longer U$2G$2.MII1_TXD1
- net MII1_TXD2: now also U1D.MII1_TXD2; no longer U$2G$2.MII1_TXD2
- net MII1_TXD3: now also U1D.MII1_TXD3
- net MII1_TXEN: now also U1D.MII1_TX_EN; no longer U$2G$2.MII1_TXD3, U$2G$2.MII1_TX_EN
- net MMC1_CLK: now also U1C.GPMC_CSN1; no longer U$2G$1.GPMC_CSN1
- net MMC1_CMD: now also U1C.GPMC_CSN2; no longer U$2G$1.GPMC_CSN2
- net MMC1_DAT0: now also U1C.GPMC_AD0; no longer U$2G$1.GPMC_AD00
- net MMC1_DAT1: now also U1C.GPMC_AD1; no longer U$2G$1.GPMC_AD01
- net MMC1_DAT2: now also U1C.GPMC_AD2; no longer U$2G$1.GPMC_AD02
- net MMC1_DAT3: now also U1C.GPMC_AD3; no longer U$2G$1.GPMC_AD03
- net MMC1_DAT4: now also U1C.GPMC_AD4; no longer U$2G$1.GPMC_AD04
- net MMC1_DAT5: now also U1C.GPMC_AD5; no longer U$2G$1.GPMC_AD05
- net MMC1_DAT6: now also U1C.GPMC_AD6; no longer U$2G$1.GPMC_AD06
- net MMC1_DAT7: now also U1C.GPMC_AD7; no longer U$2G$1.GPMC_AD07
- net N$1: now also U1A.PMIC_POWER_EN, U1A.PMIC_PWR_EN; no longer TP1.TP, U$2G$2.UART0_TXD
- net N$121: now also U1A.PMIC_LDO_PGOOD, U1A.RTC_PWRONRSTN; no longer TP2.TP, U$2G$2.UART0_RXD
- net N$172: now also R138.2, U$2.BRB; no longer C144.2, R149.1, U$2G$1.OSC1_IN, Y2.P$1
- net N$173: now also R139.2, U$2.BRA; no longer C145.2, R149.2, U$2G$1.OSC1_OUT, Y2.P$2
- net N$174: now also EEPROM_WP.TP, U1A.EEPROM_WP; no longer C144.1, C145.1, U$2G$1.OSC1_GND
- net N$175: no longer U$2G$1.TRSTN
- net N$176: now also U1B.OSC0_IN; no longer U$2G$1.OSC0_IN
- net N$177: now also U1B.OSC0_GND; no longer U$2G$1.OSC0_GND
- net N$178: now also U1C.GPMC_A11; no longer U$2G$2.MCASP0_FSR
- net N$179: now also U1A.PMIC_PB_IN; no longer U$2G$3.PMIC_IN_PB_IN
- net N$184: now also U1B.OSC0_OUT; no longer U$2G$1.OSC0_OUT
- net N$185: now also C144.1, R140.1, U$2.AIN_IREF; no longer TP3.TP, U$2G$2.UART0_CTSN
- net N$186: now also U1C.GPMC_A0; no longer TP4.TP, U$2G$2.UART0_RTSN
- net N$210: now also SV2.5, U1C.UART0_TXD; no longer R126.2, U$2G$2.LCD_PCLK
- net SERVO_0: no longer U$2G$1.GPMC_A02
- net SERVO_1: no longer U$2G$1.GPMC_A03
- net STEP_A: now also U1C.MMC0_DAT1
- net STEP_E: now also U1C.MCASP0_AXR1; no longer U$2G$1.GPMC_BEN1
- net STEP_H: now also U1C.MMC0_DAT3; no longer U$2G$1.GPMC_AD13
- net STEP_X: now also U$2.REFL_STEP, U1C.MCASP0_ACLKX; no longer U$2G$1.GPMC_AD11
- net STEP_Y: now also U1C.MCASP0_AXR0; no longer U$2G$1.GPMC_AD12
- net STEP_Z: now also U1C.MCASP0_ACLKR; no longer U$2G$1.GPMC_AD09
- net SYS_5V: now also SYS_5V.TP, U1A.SYS_VOUT@1, U1A.SYS_VOUT@2, U1A.SYS_VOUT@3, U1A.SYS_VOUT@4; no longer U$2G$3.SYS_VOUT_W4, U$2G$3.SYS_VOUT_Y4
- net SYS_RESETN: no longer IC28A.O, U$2G$1.WARMRSTN
- net TERM_A: now also U1B.AIN3; no longer U$2G$2.AIN3
- net TERM_E: now also U1B.AIN0; no longer U$2G$2.AIN0
- net TERM_H: now also U1B.AIN2; no longer U$2G$2.AIN2
- net TERM_HBP: now also U1B.AIN1; no longer U$2G$2.AIN1
- net TX0+: now also U$12.IO4, U$12.NC5; no longer U$8.TMDS.CH2+
- net TX0-: now also U$12.IO3, U$12.NC4; no longer U$8.TMDS.CH2-
- net TX1+: now also U$11.IO2, U$11.NC2; no longer U$10.TMDS.CH1+
- net TX1-: now also U$11.IO1, U$11.NC1; no longer U$10.TMDS.CH1-
- net TX2+: now also U$11.IO4, U$11.NC5; no longer U$10.TMDS.CH2+
- net TX2-: now also U$11.IO3, U$11.NC4; no longer U$10.TMDS.CH2-
- net TXC+: now also U$12.IO2, U$12.NC2; no longer U$8.TMDS.CH1+
- net TXC-: now also U$12.IO1, U$12.NC1; no longer U$8.TMDS.CH1-
- net USB0_DM: now also U1B.USB0_DM; no longer U$2G$2.USB0_DM
- net USB0_DP: now also U1B.USB0_DP; no longer U$2G$2.USB0_DP
- net USB0_ID: now also U1B.USB0_ID; no longer U$2G$2.USB0_ID
- net USB1_DM: now also U1B.USB1_DM; no longer U$2G$2.USB1_DM
- net USB1_DP: now also U1B.USB1_DP; no longer U$2G$2.USB1_DP
- net USB1_OCN: now also U1C.GPMC_A10; no longer U$2G$1.GPMC_A10
- net USB_DC: now also U1A.VIN_USB@1, U1A.VIN_USB@2, U1A.VIN_USB@3, U1B.USB0_VBUS; no longer U$2G$2.USB0_VBUS, U$2G$3.VIN_USB_Y8, U$2G$3.VIN_USB_Y9
- net USR0: now also U1C.GPMC_A5; no longer U$2G$1.GPMC_A05
- net USR1: now also U1C.GPMC_A6; no longer U$2G$1.GPMC_A06
- net USR2: now also U1C.GPMC_A7; no longer U$2G$1.GPMC_A07
- net USR3: now also U1C.GPMC_A8; no longer U$2G$1.GPMC_A08
- net VDD_ADC: now also U1B.SYS_ADC_1P8V, U1B.VREFP; no longer U$2G$2.SYS_ADC_1P8V_A4, U$2G$2.SYS_ADC_1P8V_A5, U$2G$2.VREFP
- net XDMA_EVENT_INTR0: now also U1C.XDMA_EVENT_INTR0; no longer U$2G$1.XDMA_EVENT_INTR0
- net X_A1: now also U$2.OA1; no longer IC1.OA1
- net X_A2: now also U$2.OA2; no longer IC1.OA2
- net X_B1: now also U$2.OB1; no longer IC1.OB1
- net X_B2: now also U$2.OB2; no longer IC1.OB2
Other:
- note added: "SIP LCD + LAN"
- note removed: "EEPROM"
- moved on the sheet: C102, C106, C107, C144, C145, C146, C147, C151, C152, C57, C58, C59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

Commit message: New Step down, moved some stuff around
Parts:
- removed C49: 10nF, rcl:C-EUC0402
- removed C51: 1nF, rcl:C-EUC0402
- removed D6: MBRA340T3, diode:MBRA340T3
- removed R26: 39K, rcl:R-EU_R0402
- removed U6: RT8268, SparkFun:RT8268
- removed X23: 22-05-7038-03, con-molex:22-05-7038-03
- removed X27: MINI-USB_SHIELD5P4-32005-400, con-cypressindustries:MINI-USB_SHIELD5P4-32005-400
- added U$10: TPS54202, Texas Instruments_By_element14_Batch_1:TPS54202
- added U$8: USB-MICRO, Manga_screen_rev_B-3:USB-MICRO
Connections:
- net N$106 renamed FAULT_X1
- net N$161 renamed FAULT_X0
- removed net DALLAS_W1: X23-2.S
- removed net N$189: U1C.GPMC_A2
- removed net N$25: C50.2, D6.C, L1.P$2, U6.SW
- removed net N$88: C51.1, U6.COMP
- removed net N$97: C51.2, R26.1
- net +24V: now also U$10.VIN; no longer U6.VIN
- net +3V3: no longer X23-1.S
- net D+: now also U$8.3; no longer X27G$1.3
- net D-: now also U$8.2; no longer X27G$1.2
- net ENABLE_X: now also U$2.DRV_ENN_CFG6
- net GND: now also U$10.GND, U$2.CLK, U$2.ENCN_DCO, U$8.5; no longer C49.2, D6.A, R26.2, U6.EP, U6.GND, X23-3.S, X27G$1.5
- net HEATER_E: now also U1C.GPMC_A2; no longer U11.LED5
- net ID: now also U$8.4; no longer X27G$1.4
- net N$23: now also U$10.FB; no longer U6.FB
- net N$60: now also C50.2, L1.P$2, U$10.SW; no longer C49.1, U6.SS
- net N$73: now also U$10.BOOT; no longer U6.BOOT
- net USB_DC: now also U$8.1; no longer X27G$1.1
Other:
- note removed: "Dallas 1W"
- moved on the sheet: R22

Commit message: Working on the LAN layout
Parts:
- removed C106, C17, C19, C20, C22, C24, C27, C29, C31, C34, C43, C71: 0.1uF, rcl:C-EUC0402
- removed C116, C117, C118, C119, C120, C121, C122, C123, C124, C125, C126, C127, C128, C129, C130, C131: 47pF, rcl:C-EUC0402
- removed C139, C144, C145, C18, C21, C25, C36, C52, C62, C75, C76, C77, C78, C79, C81: 4.7uF, rcl:C-EUC0402
- removed C50: 10nF, rcl:C-EUC0402
- removed C90: 10uF, rcl:C-EUC0805
- removed C96: 100uF, Panasonic-EEEFK_EEEFP:C
- removed IC1, IC12, IC15, IC2, IC24, IC5: TMC2100-LA, we-chip:TMC2100-LA
- removed IC31: CY7C65632, Revolve:CY7C65632
- removed R147: 0, DNI, rcl:R-EU_R0402
- removed R148: 0, rcl:R-EU_R0402
- removed R151: 10K, rcl:R-EU_R0402
- removed R153: 22R, rcl:R-EU_R0402
- removed R54, R86: 4.7K, rcl:R-EU_R0402
- removed R91: 33, rcl:R-EU_R0402
- removed U11: PCA9685PW, custom:PCA9685PW
- added C13: 0.1uF, rcl:C-EUC0402
- added C5: 18pF, rcl:C-EUC0402
- added H1, H2, H3, H4: MOUNT-HOLE3.2, holes:MOUNT-HOLE3.2
- added J1: (no value), OSD3358-SM-RED Platform:CTI-JTAG
- added Q9: MMBT2907, OSD3358-SM-RED Platform:MMBT2907SMD
- added R143, R144: 4.7K, rcl:R-EU_R0402
- added R26: 1M, rcl:R-EU_R0402
- added SV3: (no value), con-lstb:MA04-2
- added SV4: (no value), con-lstb:MA03-1
- added SV5: (no value), con-lstb:MA04-1
- added U$13, U$14, U$15, U$16: TRINAMIC_TMC2130_QFN36, TMC2130-Eval_v13:TRINAMIC_TMC2130_QFN36
- added U2: TUSB2046BIRHBT, Texas Instruments_By_element14_Batch_1:TUSB2046BIRHBT
- added U3, U4: TPD2E001DRSR, Texas Instruments_By_element14_Batch_1:TPD2E001DRSR
- added U5: SN74HC245DW, Texas Instruments_By_element14_Batch_1:SN74HC245DW
- added U7: TLVH431, OSD3358-SM-RED Platform:TLVH431
- added Y5: ABS07-32.768KHZ-T, OSD3358-SM-RED Platform:ABS07-32.768KHZ-T
- C1: value 22nF -> 0.1uF; MPN C1005X7R1E223K050BB -> CL10B104KB8NNND
- C12: value 4.7uF -> 0.1uF; MPN GRM155R60J475ME47D -> CL10B104KB8NNND
- C138, C140, C141, C142: value 4.7uF -> 0.1uF
- C143: value 4.7uF -> 10uF
- C48, C80: value 10uF -> 22uF
- C6: value 0.1uF -> 18pF; MPN CL10B104KB8NNND -> GRM155R60J475ME47D
- EEPROM_WP, PMIC_NRESET, SYS_5V, SYS_RTC_1V8, SYS_VDD1_3V3, SYS_VDD2_3V3, SYS_VDD3_3V3, VDDS_DDR, VDDS_PLL, VDD_CODE, VDD_MPU: value TPPAD1-13 -> TPB1,27; device testpad:TPPAD1-13 -> testpad:TPB1,27
- R1: value 0.1R -> 1.5K; device rcl:R-EU_R0805 -> rcl:R-EU_R0402; MPN RL1220S-R10-F -> RC0402FR-0710KL
- R12: value 44.3K,1% -> 100K,1%; MPN RC1005F4422CS -> (none)
- R152: value 10K -> 10K,1%
- R2: value 0.1R -> 0,DNI; device rcl:R-EU_R0805 -> rcl:R-EU_R0402; MPN RL1220S-R10-F -> RC0402JR-074K7L
- R22: value 10K,1% -> 13.3K,1%
- R24: value 4.7K -> 0R,DNI
- R41: value 10K -> 10K, 1%; device rcl:R-EU_R0402 -> OSD3358-SM-RED Platform:R-US_R0402; MPN RC0402FR-0710KL -> (none)
- R49: value 10K -> 40.2K, 1%; device rcl:R-EU_R0402 -> OSD3358-SM-RED Platform:R-US_R0402; MPN RC0402FR-0710KL -> (none)
- R53: value 2.2R -> 499; device rcl:R-EU_R0402 -> OSD3358-SM-RED Platform:R-US_R0402; MPN RC1005J2R2CS -> (none)
- R87: value 650R, 1% -> 4.7K
- SV2: device con-lstb:MA05-1 -> con-lstb:MA04-2
- U$2: MPN (none) -> TMC2130-LA
- U$9: value SN74AUC1G74DCTR -> TRINAMIC_TMC2130_QFN36; device Revolve:SN74AUC1G74DCTR -> TMC2130-Eval_v13:TRINAMIC_TMC2130_QFN36
- U1: MPD (none) -> OSD3358-512M-BAS000
- Y1: value 24MHz -> 25MHz
- Y4: value 12 MHz -> 6 MHz
Connections:
- net N$1 renamed PMIC_PWR_EN
- net N$103 renamed PMIC_SCL
- net N$104 renamed PMIC_SDA
- net N$121 renamed PMIC_LDO_PGOOD
- net N$143 renamed PMIC_NWAKEUP
- net N$144 renamed PMIC_NINT
- net N$157 renamed TXP
- net N$158 renamed TXN
- net N$159 renamed RXP
- net N$160 renamed RXN
- net N$174 renamed EEPROM_WP
- removed net 12MHZ: R91.1, U$7.OSC_IN/AP3
- removed net D+: U$8.3, U10.D+
- removed net D-: U$8.2, U10.D-
- removed net ENABLE_A: IC24.DRV_ENN_CFG6
- removed net ENABLE_E: IC12.DRV_ENN_CFG6
- removed net ENABLE_H: IC15.DRV_ENN_CFG6
- removed net ENABLE_X: IC1.DRV_ENN_CFG6, U$2.DRV_ENN_CFG6
- removed net ENABLE_Y: IC2.DRV_ENN_CFG6
- removed net ENABLE_Z: IC5.DRV_ENN_CFG6
- removed net END_STOP_X_1: U19.G=A
- removed net END_STOP_X_2: U19.J=D
- removed net END_STOP_Y_1: U19.H=B
- removed net END_STOP_Y_2: U19.K=E
- removed net END_STOP_Z_1: U19.I=C
- removed net END_STOP_Z_2: U19.L=F
- removed net FAULT_X0: U$2.SWN_DIAG0
- removed net FAULT_X1: U$2.SWP_DIAG1
- removed net I2C2_SCL: U11.SCL
- removed net I2C2_SDA: U11.SDA
- removed net ID: U$8.4, U10.ID
- removed net IREF_A_RAW: R73.2, U11.LED2
- removed net IREF_E_RAW: R60.2, U11.LED14
- removed net IREF_H1: C81.1, R43.2, R73.1
- removed net IREF_H_RAW: R31.2, U11.LED15
- removed net IREF_X1: C145.1, R140.2, R141.1
- removed net IREF_X_RAW: R141.2, R41.2, U11.LED11
- removed net IREF_Y_RAW: R37.2, U11.LED12
- removed net IREF_Z_RAW: R58.2, U11.LED13
- removed net N$100: IC15.SDO_NAO_CFG0
- removed net N$101: IC15.ENCB_DCEN_CFG4
- removed net N$102: IC15.ENCA_DCIN_CFG5
- removed net N$105: SYS_VDD1_3V3.TP, U1A.SYS_VDD1_3P3V@1, U1A.SYS_VDD1_3P3V@2, U1A.SYS_VDD1_3P3V@3, U1A.SYS_VDD1_3P3V@4
- removed net N$107: C70.1, IC15.VCC, R52.2
- removed net N$108: C71.1, IC1.VCC, R53.2
- removed net N$110: C72.1, IC2.VCC, R59.2
- removed net N$111: C74.1, IC12.VCC, R71.2
- removed net N$112: IC12.OA2, X17-1.S
- removed net N$119: IC15.OA2, X18-1.S
- removed net N$120: SYS_VDD3_3V3.TP, U1A.SYS_VDD3_3P3V@1, U1A.SYS_VDD3_3P3V@2, U1A.SYS_VDD3_3P3V@3, U1A.SYS_VDD3_3P3V@4, U1A.SYS_VDD3_3P3V@5, U1A.SYS_VDD3_3P3V@6, U1A.SYS_VDD3_3P3V@7, U1A.SYS_VDD3_3P3V@8
- removed net N$131: C52.1, IC24.AIN_IREF, R43.1
- removed net N$133: IC24.SCK_CFG2
- removed net N$135: IC24.OA1, X25-2.S
- removed net N$136: C55.2, IC24.5VOUT, R72.1
- removed net N$138: IC24.SDI_NAI_CFG1
- removed net N$139: IC24.SDO_NAO_CFG0
- removed net N$140: IC24.ENCB_DCEN_CFG4
- removed net N$141: IC24.ENCA_DCIN_CFG5
- removed net N$142: SYS_RTC_1V8.TP, U1A.SYS_RTC_1P8V@1, U1A.SYS_RTC_1P8V@2
- removed net N$146: U1A.VDDSHV1, U1A.VDDSHV2, U1A.VDDSHV3, U1A.VDDSHV4, U1A.VDDSHV5, U1A.VDDSHV6
- removed net N$148: IC24.OA2, X25-1.S
- removed net N$165: U1C.GPMC_CLK
- removed net N$166: C86.2, R126.1, U$2.5VOUT
- removed net N$175: R86.2
- removed net N$178: U1C.GPMC_A11
- removed net N$18: IC1.BRB, R1.2
- removed net N$185: C144.1, R140.1, U$2.AIN_IREF
- removed net N$186: U1C.GPMC_A0
- removed net N$187: C155.1, IC31.VCC, R147.1, R148.1
- removed net N$188: U1C.GPMC_A1
- removed net N$190: U1C.GPMC_A3
- removed net N$191: IC31.VCC_A, IC31.VCC_A@1, IC31.VCC_A@2, IC31.VCC_D, IC31.VREG
- removed net N$197: IC31.DD+[3], U$6.D+@0
- removed net N$198: IC31.DD–[3], U$6.D-@0
- removed net N$199: IC31.DD+[4], U$6.D+@1
- removed net N$200: IC31.DD–[4], U$6.D-@1
- removed net N$202: U$9.D, U$9.NQ
- removed net N$205: R91.2, U$9.Q
- removed net N$210: SV2.5, U1C.UART0_TXD
- removed net N$213: C157.2, IC31.XOUT, Y4.P$1
- removed net N$215: SV2.4, U1C.UART0_RXD
- removed net N$26: C25.1, IC5.AIN_IREF, R27.1
- removed net N$31: C21.2, IC1.5VOUT, R53.1
- removed net N$47: C33.2, IC2.5VOUT, R59.1
- removed net N$50: IC5.OA1, X16-2.S
- removed net N$51: C37.2, IC5.5VOUT, R70.1
- removed net N$53: IC2.SDO_NAO_CFG0
- removed net N$54: IC5.SDI_NAI_CFG1
- removed net N$55: IC5.SDO_NAO_CFG0
- removed net N$56: IC2.ENCB_DCEN_CFG4
- removed net N$57: IC5.ENCB_DCEN_CFG4
- removed net N$58: IC5.ENCA_DCIN_CFG5
- removed net N$60: C50.2, L1.P$2, U$10.SW
- removed net N$65: IC2.ENCA_DCIN_CFG5
- removed net N$73: C50.1, U$10.BOOT
- removed net N$74: C62.1, IC12.AIN_IREF, R35.1
- removed net N$76: IC12.SCK_CFG2
- removed net N$78: IC12.OA1, X17-2.S
- removed net N$79: C65.2, IC12.5VOUT, R71.1
- removed net N$81: IC12.SDI_NAI_CFG1
- removed net N$82: IC12.SDO_NAO_CFG0
- removed net N$83: IC12.ENCB_DCEN_CFG4
- removed net N$84: IC12.ENCA_DCIN_CFG5
- removed net N$89: C36.1, IC15.AIN_IREF, R50.1
- removed net N$91: IC15.SCK_CFG2
- removed net N$94: IC15.OA1, X18-2.S
- removed net N$95: C68.2, IC15.5VOUT, R52.1
- removed net N$99: IC15.SDI_NAI_CFG1
- removed net SPI0_CS0: U1C.SPI0_CS0
- removed net SPI0_CS1: U1C.SPI0_CS1
- removed net USB1_OCN: U1C.GPMC_A10
- removed net XDMA_EVENT_INTR0: U$9.CLK, U1C.XDMA_EVENT_INTR0
- removed net X_CFG1: IC1.SDI_NAI_CFG1
- removed net X_CFG2: IC1.SCK_CFG2
- new net 5VIN_Y: C72.1, R59.2, U$13.VCC
- new net 5VOUT_A: C55.2, R72.1, R73.2, U$16.5VOUT
- new net 5VOUT_E: C65.2, R35.2, R71.1, U$14.5VOUT
- new net 5VOUT_H: C68.2, R31.2, R52.1, U$15.5VOUT
- new net 5VOUT_X: C86.2, R126.1, R140.2, U$2.5VOUT
- new net 5VOUT_Y: C33.2, R37.2, R59.1, U$13.5VOUT
- new net 5VOUT_Z: C37.2, R27.2, R70.1, U$9.5VOUT
- new net CLKOUT1_25MHZ: R2.1, U1C.XDMA_EVENT_INTR0
- new net CLKOUT2_48MHZ: U1C.XDMA_EVENT_INTR1, U2.TSTPLL/48MCLK
- new net ECAP1: SV5.3, U1C.UART0_TXD
- new net ECAP2: SV5.2, U1C.UART0_RXD
- new net EHRPWM1A: U1C.GPMC_A2, U5.A5
- new net EHRPWM1B: U1C.GPMC_A3, U5.A6
- new net EHRPWM2A: U1C.GPMC_AD8, U5.A7
- new net EHRPWM2B: U1C.GPMC_AD9, U5.A8
- new net EMU0: J1.EMU0, U1B.EMU0
- new net EMU1: J1.EMU1, U1B.EMU1
- new net ENABLE_B: SV2.4
- new net ENABLE_C: SV3.3
- new net END_STOP_X1: U19.G=A, U1C.GPMC_BEN1
- new net END_STOP_X2: U19.J=D, U1C.GPMC_A1
- new net END_STOP_Y1: U19.H=B, U1C.GPMC_A11
- new net END_STOP_Y2: U19.K=E, U1C.GPMC_CSN0
- new net END_STOP_Z1: U19.I=C, U1C.GPMC_AD14
- new net END_STOP_Z2: U19.L=F, U1C.GPMC_AD15
- new net FAULT_A: R44.1, U$16.SWN_DIAG0, U$16.SWP_DIAG1
- new net FAULT_B: SV2.2
- new net FAULT_C: SV3.1
- new net GPIO0_18: U1B.USB0_DRVVBUS
- new net GPIO0_26: U1C.GPMC_AD10
- new net I2C1_SCL: U1C.UART1_TXD
- new net I2C1_SDA: U1C.UART1_RXD
- new net N$1: R41.1, R49.2, U7.REF
- new net N$25: R152.1, U1A.RTC_KALDO_ENN
- new net QUAD_ENCODER_A: U1C.GPMC_A4
- new net QUAD_ENCODER_B: U1C.GPMC_A5
- new net SPI0_CSA: U$16.CSN_CFG3, U1D.RMII1_REF_CLK
- new net SPI0_CSE: U$14.CSN_CFG3, U1C.GPMC_A0
- new net SPI0_CSH: U$15.CSN_CFG3, U1C.GPMC_CSN3
- new net SPI0_CSY: U$13.CSN_CFG3, U1C.SPI0_CS1
- new net SPI0_CSZ: U$9.CSN_CFG3, U1C.GPMC_CLK
- new net SPI1_CS0: SV3.4, U1C.UART1_CTSN
- new net SPI1_CS1: SV2.3, U1C.UART1_RTSN
- new net SPI1_MISO: SV2.6, SV3.6, U1C.UART0_CTSN
- new net SPI1_MOSI: SV2.8, SV3.8, U1C.UART0_RTSN
- new net SPI1_SCLK: SV2.1, SV3.2, U1C.ECAP0_IN_PWM0_OUT
- new net SW: C2.1, L1.P$2, U$10.SW
- new net SYS_RTC_1V8: Q9.C, R49.1, SYS_RTC_1V8.TP, U1A.SYS_RTC_1P8V@1, U1A.SYS_RTC_1P8V@2, U7.ANODE
- new net SYS_VDD1_3V3: C13.1, C140.1, C141.1, C142.1, C143.1, C150.1, C155.1, IC29.VDDIO, IC30.VCC@0, IC30.VCC@1, IC30.VCC@2, IC30.VCC@3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
- new net SYS_VDD3_3V3: Q9.E, R41.2, R53.2, SYS_VDD3_3V3.TP, U1A.SYS_VDD3_3P3V@1, U1A.SYS_VDD3_3P3V@2, U1A.SYS_VDD3_3P3V@3, U1A.SYS_VDD3_3P3V@4, U1A.SYS_VDD3_3P3V@5, U1A.SYS_VDD3_3P3V@6, U1A.SYS_VDD3_3P3V@7, U1A.SYS_VDD3_3P3V@8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
- new net TCK: J1.TCK, U1B.TCK
- new net TDI: J1.TDI, U1B.TDI
- new net TDO: J1.TDO, U1B.TDO
- new net TIMER4: U1C.GPMC_ADVN_ALE, U5.A1
- new net TIMER5: U1C.GPMC_BEN0_CLE, U5.A2
- new net TIMER6: U1C.GPMC_WEN, U5.A3
- new net TIMER7: U1C.GPMC_OEN_REN, U5.A4
- new net TK_A: U1B.AIN7
- new net TK_E: U1B.AIN4
- new net TK_H: U1B.AIN5
- new net TK_HBP: U1B.AIN6
- new net TMS: J1.TMS, U1B.TMS
- new net TRSRTN: J1.TRSTN
- new net TRSTN: U1B.TRSTN
- new net UART4_RXD: SV4.1, U1C.GPMC_WAIT0
- new net UART4_TXD: SV4.2, U1C.GPMC_WPN
- new net USB1_DM3: U$6.D-@0, U2.DM3, U4.IO1
- new net USB1_DM4: U$6.D-@1, U2.DM4, U3.IO1
- new net USB1_DP3: U$6.D+@0, U2.DP3, U4.IO2
- new net USB1_DP4: U$6.D+@1, U2.DP4, U3.IO2
- new net USB_HOST_5V: U$5.VBUS@0, U$5.VBUS@1, U$6.VBUS@0, U$6.VBUS@1
- new net USB_XTAL1: C157.2, U2.XTAL1, Y4.P$1
- new net VCC_E: C74.1, R71.2, U$14.VCC
- new net VCC_H: C70.1, R52.2, U$15.VCC
- new net VIN_BAT: U1A.VIN_BAT@1, U1A.VIN_BAT@2, U1A.VIN_BAT@3
- net +24V: now also C1.2, U$13.VS, U$13.VSA, U$14.VS, U$14.VSA, U$15.VS, U$15.VSA, U$16.VS, U$16.VSA, U$9.VS, U$9.VSA; no longer C19.1, C20.2, C22.2, C24.1, C27.1, C29.1, C31.1, C34.1, C43.1, C6.1, C90.1, C96.+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
- net +3V3: now also R143.1, R144.1, U$13.VCC_IO, U$14.VCC_IO, U$15.VCC_IO, U$16.VCC_IO, U$9.VCC_IO; no longer C106.1, C2.1, IC1.VCC_IO, IC12.VCC_IO, IC15.VCC_IO, IC2.VCC_IO, IC24.VCC_IO, IC5.VCC_IO, R24.2, R54.2, U$9.NCLR, U$9.NPRE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
- net +5V: no longer R147.2
- net CGND: now also U$3.SHD1, U$3.SHD2, U$5.SHD1, U$5.SHD2, U$5.SHD3, U$5.SHD4, U$6.SHD1, U$6.SHD2, U$6.SHD3, U$6.SHD4, U$8.GND@0, U$8.GND@1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
- net DIR_A: now also U$16.REFR_DIR; no longer IC24.REFR_DIR
- net DIR_B: now also SV2.5
- net DIR_C: now also SV3.5
- net DIR_E: now also U$14.REFR_DIR; no longer IC12.REFR_DIR
- net DIR_H: now also U$15.REFR_DIR; no longer IC15.REFR_DIR
- net DIR_X: no longer IC1.REFR_DIR
- net DIR_Y: now also U$13.REFR_DIR; no longer IC2.REFR_DIR
- net DIR_Z: now also U$9.REFR_DIR; no longer IC5.REFR_DIR
- net EMMC_RST: no longer U1C.GPMC_A4
- net ENABLE: now also U5.~OE; no longer U11.~OE
- net FAN0: now also U5.B5; no longer U11.LED7
- net FAN1: now also U5.B6; no longer U11.LED8
- net FAN2: now also U5.B7; no longer U11.LED9
- net FAN3: now also U5.B8; no longer U11.LED10
- net FAULT_E: now also U$14.SWN_DIAG0, U$14.SWP_DIAG1; no longer IC12.SWN_DIAG0
- net FAULT_H: now also U$15.SWN_DIAG0, U$15.SWP_DIAG1; no longer IC15.SWN_DIAG0, IC24.SWN_DIAG0, R44.1
- net FAULT_X: now also R143.2, U$2.SWN_DIAG0, U$2.SWP_DIAG1, U1C.GPMC_AD11; no longer IC1.SWN_DIAG0, R54.1
- net FAULT_Y: now also R144.2, U$13.SWN_DIAG0, U$13.SWP_DIAG1; no longer IC2.SWN_DIAG0, R24.1
- net FAULT_Z: now also U$9.SWN_DIAG0, U$9.SWP_DIAG1; no longer IC5.SWN_DIAG0
- net GND: now also C1.1, C13.2, J1.GND1, J1.GND2, J1.GND3, J1.GND4, J1.GND5, R141.1, R152.2, R43.1, R50.1, R58.1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; no longer C106.2, C116.2, C117.2, C118.2, C119.2, C120.2, C121.2, C122.2, C123.2, C124.2, C125.2, C126.2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
- net HDMI_1V8: now also C12.1
- net HDMI_INT: now also U1C.GPMC_A10; no longer U1C.GPMC_A9
- net HEATER_A: now also U5.B4; no longer U11.LED6
- net HEATER_E: now also U5.B1; no longer U1C.GPMC_A2
- net HEATER_H: now also U5.B2; no longer U11.LED3
- net HEATER_HBP: now also U5.B3; no longer U11.LED4
- net IREF_E: now also R35.1, R60.2, U$14.AIN_IREF; no longer C79.1, R35.2, R60.1
- net IREF_H: now also U$15.AIN_IREF; no longer C75.1
- net IREF_X: now also R140.1, R141.2, U$2.AIN_IREF; no longer C77.1, R41.1, R49.2
- net IREF_Y: now also U$13.AIN_IREF; no longer C76.1
- net IREF_Z: now also R27.1, R58.2, U$9.AIN_IREF; no longer C78.1, R27.2, R58.1
- net LCD_D0: no longer C116.1
- net LCD_D1: no longer C117.1
- net LCD_D10: no longer C126.1
- net LCD_D11: no longer C127.1
- net LCD_D12: no longer C128.1
- net LCD_D13: no longer C129.1
- net LCD_D14: no longer C130.1
- net LCD_D15: no longer C131.1
- net LCD_D2: no longer C118.1
- net LCD_D3: no longer C119.1
- net LCD_D4: no longer C120.1
- net LCD_D5: no longer C121.1
- net LCD_D6: no longer C122.1
- net LCD_D7: no longer C123.1
- net LCD_D8: no longer C124.1
- net LCD_D9: no longer C125.1
- net LCD_DE: no longer R153.2
- net LCD_PCLK: no longer R153.1
- net N$109: now also U$9.VCC; no longer IC5.VCC
- net N$113: now also U$15.OB1; no longer IC15.OB1
- net N$12: now also U$15.CPO; no longer IC15.CPO
- net N$126: now also U$16.BRB; no longer IC24.BRB
- net N$128: now also U$16.BRA; no longer IC24.BRA
- net N$13: now also U$15.BRB; no longer IC15.BRB
- net N$132: now also U$16.CPI; no longer IC24.CPI
- net N$134: now also U$16.OB2; no longer IC24.OB2
- net N$137: now also U$16.VCP; no longer IC24.VCP
- net N$14: now also U$9.CPO; no longer IC5.CPO
- net N$145: now also U$16.VCC; no longer IC24.VCC
- net N$147: now also U$16.OB1; no longer IC24.OB1
- net N$15: now also U$9.BRB; no longer IC5.BRB
- net N$16: now also U$9.OA2, X16-2.S; no longer C1.1, IC1.CPI
- net N$17: now also U2.~OVRCUR1, U2.~OVRCUR2, U2.~OVRCUR3, U2.~OVRCUR4; no longer C1.2, IC1.CPO
- net N$180: now also R2.2
- net N$19: now also U$13.OA2, X15-2.S; no longer IC1.BRA, R2.2
- net N$192: now also R24.2, U2.TSTMODE; no longer IC31.RREF
- net N$193: now also U2.DP1; no longer IC31.DD+[1]
- net N$194: now also U2.DM1; no longer IC31.DD–[1]
- net N$195: now also U2.DP2; no longer IC31.DD+[2]
- net N$196: now also U2.DM2; no longer IC31.DD–[2]
- net N$2: now also U$13.OB1; no longer IC2.OB1
- net N$20: now also U$13.OA1, X15-1.S; no longer C12.1, IC1.AIN_IREF, R49.1
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Other:
- note added: "Ext driver B"
- note added: "Ext driver C"
- note removed: "PWM extension"
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
Commit message: Working on layout
Parts:
- removed C5, C6: 18pF, rcl:C-EUC0402
- removed R26, R84: 1M, rcl:R-EU_R0402
- removed U5: SN74HC245DW, Texas Instruments_By_element14_Batch_1:SN74HC245DW
- removed Y3: 25 MHz, Revolve:445C33D24M0000011.4X4.7
- removed Y5: ABS07-32.768KHZ-T, OSD3358-SM-RED Platform:ABS07-32.768KHZ-T
- added Y2: 25MHz, Revolve:445C33D24M00000SMALL
Connections:
- removed net +3V3: C23.1, C30.1, C44.1, C53.1, C61.1, C63.1, C84.1, R114.2, R117.2, R118.2, R119.2, R120.2, R143.1, R144.1, R28.2, R36.2, R44.2, R51.2, U$13.VCC_IO, U$14.VCC_IO, U$15.VCC_IO, U$16.VCC_IO, U$2.VCC_IO, U$9.VCC_IO, U19.VCC
- removed net ENABLE: U5.~OE
- removed net N$33: C5.1, C6.1, U1B.OSC1_GND
- removed net N$42: C6.2, R26.2, U1B.OSC1_OUT, Y5.P$2
- removed net N$43: C5.2, R26.1, U1B.OSC1_IN, Y5.P$1
- net EHRPWM1A: no longer U5.A5
- net EHRPWM1B: no longer U5.A6
- net EHRPWM2A: no longer U5.A7
- net EHRPWM2B: no longer U5.A8
- net FAN0: no longer U5.B5
- net FAN1: no longer U5.B6
- net FAN2: no longer U5.B7
- net FAN3: no longer U5.B8
- net GND: now also X11-3.S, X7-3.S, X8-3.S; no longer U5.GND
- net HEATER_A: no longer U5.B4
- net HEATER_E: no longer U5.B1
- net HEATER_H: no longer U5.B2
- net HEATER_HBP: no longer U5.B3
- net N$151: now also X11-2.S
- net N$180: now also Y2.P$2; no longer R84.2, Y3.P$2
- net N$181: now also Y2.P$1; no longer Y3.P$1
- net N$183: no longer R84.1
- net N$237: now also X8-2.S
- net N$241: now also X7-2.S
- net SYS_5V: no longer U5.DIR, U5.VCC
- net SYS_VDD1_3V3: now also C23.1, C30.1, C44.1, C53.1, C61.1, C63.1, C84.1, R114.2, R117.2, R118.2, R119.2, R120.2, R143.1, R144.1, R28.2, R36.2, R44.2, R51.2, U$13.VCC_IO, U$14.VCC_IO, U$15.VCC_IO, U$16.VCC_IO, U$2.VCC_IO, U$9.VCC_IO, U19.VCC
- net TIMER4: no longer U5.A1
- net TIMER5: no longer U5.A2
- net TIMER6: no longer U5.A3
- net TIMER7: no longer U5.A4
