File: PCB/Revolve_A0/Revolve_A0.sch (EAGLE design)
At the start: 365 parts, among them IC29 LAN8710A, IC30 MTFC2GMDEA, IC6 74AHC1G126DCK, IC7 74AHC1G126DCK, Q1 AON6758, Q2 AON6758, Q3 AON6758, Q8 AON6758, Q9 MMBT2907, U1 OSD3358-512M-BSM, U10 TPD4S012_DRY_6, U19 CD4050BD, U2 TUSB2046BIRHBT, U3 TPD2E001DRSR, U4 TPD2E001DRSR, U7 TLVH431, X1 22-05-7038-03, X10 22-05-7038-03, X11 22-05-7038-03, X12 22-05-7048-04, X13 22-05-7038-03, X14 22-05-7048-04, X15 22-05-7048-04, X16 22-05-7048-04, X17 22-05-7048-04, X18 22-05-7048-04, X19 22-05-7038-03, X2 MSTBA4, X20 MSTBA4, X21 MSTBA2, X22 22-05-7038-03, X24 HDMI, X25 22-05-7048-04, X26 MSTBA2, X29 22-05-7038-03, X3 MSTBA2, X4 22-05-7028-02, X5 22-05-7028-02, X6 22-05-7028-02, X7 22-05-7038-03, X8 22-05-7038-03, X9 22-05-7028-02, Y1 25MHz, Y2 25MHz, Y4 6 MHz

Commit message: Almost done with schematic
Parts:
- removed C104, C105: 0.1uF, rcl:C-EUC0402
- removed F1: FUSE, fuse:FUSE
- removed FH1, FH2: FUSE-HOLDER, Replicape_Rev_B0:FUSE-HOLDER
- removed LED8: blue, led:LEDCHIP-LED0603
- removed RT1: (no value), rcl:R-US_0204/5
- removed U$11, U$12: DF10G7M1N, Revolve:DF10G7M1N
- added C14, C17: 22uF, rcl:C-EUC1206
- added C18, C19, C5, C6: 0.1uF, rcl:C-EUC0402
- added Q10, Q11, Q13, Q14: DMC2038LVT, Manga_screen_rev_B:DMC2038LVT
- added Q12: (no value), semicon-smd-ipc:NPN-TRANSISTOR_SOT23
- added R142, R54, R91: 4.7K, rcl:R-EU_R0402
- added R26: 0.001,1%, resistor:R-EU_R2512
- added R84, R86: 100K,1%, rcl:R-EU_R0402
- added U$17: SISS27DN, Revolve:SISS27DN
- added U$18: TPD12S016-RKT, Revolve:TPD12S016-RKT
- added U11: SN74AHC595PW, Replicape_B3:SN74AHC595PW
- added U5: UA78L05ACD, Texas Instruments_By_element14_Batch_1:UA78L05ACD
- added U6, U8, U9: TPD4S012_DRY_6_P1_P, OSD3358-SM-RED Platform:TPD4S012_DRY_6_P1_P
- C148, C149: value 30pF -> 18pF
- IC30: MPN (none) -> MTFC2GMDEA-0M WT
- Q4, Q5, Q6, Q7: SPN (none) -> 785-1084-1-ND
- R1: value 1.5K -> 10K
- R105, R106, R107, R108, R109, R110, R111, R112, R113, R114, R115, R117, R118, R119: value 100K -> 100K,1%; MPN RC0402JR-074K7L -> RC0402FR-07100KL
- R116, R120: value 100K -> 100K,1%; MPN RC0402JR-074K7L -> RC0402FR-07100KL; SPN (none) -> 311-100KLRCT-ND
- R12: MPN (none) -> RC0402FR-07100KL; SPN (none) -> 311-100KLRCT-ND
- R2: value 0,DNI -> 0R,DNI; MPN RC0402JR-074K7L -> RC0402JR-070RL; SPN (none) -> 311-0.0JRCT-ND
- R22: MPN RC0402FR-0710KL -> RC0402FR-0713K3L; SPN (none) -> YAG2974CT-ND
- R24: MPN RC0402JR-074K7L -> RC0402JR-070RL; SPN (none) -> 311-0.0JRCT-ND
- R45: value 4.7K -> 100K,1%; MPN RC0402JR-074K7L -> RC0402FR-07100KL; SPN (none) -> 311-100KLRCT-ND
- R55, R56, R57: value 4.7K -> 10K; MPN RC0402JR-074K7L -> RC0402FR-0710KL
- U$13, U$14, U$15, U$16, U$2, U$9: SPN (none) -> 1460-1130-2-ND
- U$5, U$6: SPN (none) -> WM4073-ND
- U$7: SPN (none) -> 568-12059-ND
- U3: value TPD2E001DRSR -> TPS2061D; device Texas Instruments_By_element14_Batch_1:TPD2E001DRSR -> Texas Instruments_By_element14_Batch_1:TPS2061D
- U4: value TPD2E001DRSR -> TPD4S012_DRY_6_P1_P; device Texas Instruments_By_element14_Batch_1:TPD2E001DRSR -> OSD3358-SM-RED Platform:TPD4S012_DRY_6_P1_P
- X24: value HDMI -> HDMI4; device hdmi:HDMI -> hdmi:HDMI4; MPN (none) -> 609-4614-2-ND
- Y1, Y2: SPN (none) -> CTX1434TR-ND
Connections:
- net N$152 renamed VDDCR
- net N$25 renamed RTC_KALDO_ENN
- net TK_HBP renamed I_MEASURE
- removed net ECAP1: SV5.3, U1C.UART0_TXD
- removed net ECAP2: SV5.2, U1C.UART0_RXD
- removed net EHRPWM1A: U1C.GPMC_A2
- removed net EHRPWM1B: U1C.GPMC_A3
- removed net EHRPWM2A: U1C.GPMC_AD8
- removed net EHRPWM2B: U1C.GPMC_AD9
- removed net GPIO0_18: U1B.USB0_DRVVBUS
- removed net GPIO0_26: U1C.GPMC_AD10
- removed net N$17: U2.~OVRCUR1, U2.~OVRCUR2, U2.~OVRCUR3, U2.~OVRCUR4
- removed net N$193: U$5.D+@0, U2.DP1
- removed net N$194: U$5.D-@0, U2.DM1
- removed net N$195: U$5.D+@1, U2.DP2
- removed net N$196: U$5.D-@1, U2.DM2
- removed net SPI0_CSE: U$14.CSN_CFG3, U1C.GPMC_A0
- removed net SPI0_CSH: U$15.CSN_CFG3, U1C.GPMC_CSN3
- removed net SPI0_CSX: U$2.CSN_CFG3, U1C.SPI0_CS0
- removed net SPI0_CSY: U$13.CSN_CFG3, U1C.SPI0_CS1
- removed net SPI0_CSZ: U$9.CSN_CFG3, U1C.GPMC_CLK
- removed net TIMER4: U1C.GPMC_ADVN_ALE
- removed net TIMER5: U1C.GPMC_BEN0_CLE
- removed net TIMER6: U1C.GPMC_WEN
- removed net TIMER7: U1C.GPMC_OEN_REN
- removed net TK_A: U1B.AIN7
- removed net USB_HOST_5V: U$5.VBUS@0, U$5.VBUS@1, U$6.VBUS@0, U$6.VBUS@1
- removed net VIN_BAT: U1A.VIN_BAT@1, U1A.VIN_BAT@2, U1A.VIN_BAT@3
- new net +12V: C5.2, U5.OUT, X12-4.S
- new net +24V_FOR_5V: C1.2, C47.1, D5.C, U$10.VIN
- new net ENABLE_STUFF: Q12.B, R91.1, U1B.USB0_DRVVBUS
- new net EN_TK_A: Q14.G1, Q14.G2, R142.2, U11.QD, X11-1.S
- new net EN_TK_E: Q10.G1, Q10.G2, R76.2, U11.QA, X29-1.S
- new net EN_TK_H: Q11.G1, Q11.G2, R92.2, U11.QB, X7-1.S
- new net EN_TK_HBP: Q13.G1, Q13.G2, R93.2, U11.QC, X8-1.S
- new net MGND: C102.2, C57.2, C58.2, C59.2, LED1.C, LED2.C, LED3.C, LED4.C, Q1.S, Q2.S, Q3.S, Q8.S, R26.2, R46.1, R47.1, R48.1, R75.1
- new net N$26: R84.2, R86.1, U$17.G
- new net N$31: U$18.HPD_B, X24.HOT_PLUG_DETECT
- new net N$33: Q10.D1, R1.1
- new net N$47: Q10.D2, R18.2
- new net N$50: Q13.D1, R56.1
- new net N$53: Q14.D1, R57.1
- new net N$55: U$18.SDA_B, X24.SDA
- new net N$56: U$18.SCL_B, X24.SCL
- new net N$57: U$18.CEC_B, X24.CEC
- new net N$58: Q11.D2, R17.2
- new net N$59: Q13.D2, R13.2
- new net N$60: Q14.D2, R77.2
- new net N$65: Q11.D1, R55.1
- new net SPI0_CS0: U$13.CSN_CFG3, U$14.CSN_CFG3, U$15.CSN_CFG3, U$16.CSN_CFG3, U$2.CSN_CFG3, U$9.CSN_CFG3, U1C.SPI0_CS0
- new net SPI0_CS1: U11.RCLK, U1C.SPI0_CS1
- new net SPI0_MISO_E: U$14.SDO_NAO_CFG0, U$15.SDI_NAI_CFG1
- new net SPI0_MISO_H: U$15.SDO_NAO_CFG0, U$16.SDI_NAI_CFG1
- new net SPI0_MISO_X: U$13.SDI_NAI_CFG1, U$2.SDO_NAO_CFG0
- new net SPI0_MISO_Y: U$13.SDO_NAO_CFG0, U$9.SDI_NAI_CFG1
- new net SPI0_MISO_Z: U$14.SDI_NAI_CFG1, U$9.SDO_NAO_CFG0
- new net USB1_DM1: U$5.D-@0, U2.DM1, U9.D+
- new net USB1_DM2: U$5.D-@1, U2.DM2, U6.D+
- new net USB1_DP1: U$5.D+@0, U2.DP1, U9.D-
- new net USB1_DP2: U$5.D+@1, U2.DP2, U6.D-
- new net USB1_DRVVBUS: U1B.USB1_DRVVBUS
- new net USB_OC: U2.~OVRCUR1, U2.~OVRCUR2, U2.~OVRCUR3, U2.~OVRCUR4, U3.~OC
- new net USB_PWR: U2.~PWRON1, U3.IN, U3.IN_2
- new net USB_VBUS: C14.1, C17.1, U$5.VBUS@0, U$5.VBUS@1, U$6.VBUS@0, U$6.VBUS@1, U3.OUT, U3.OUT_2, U3.OUT_3, U4.VBUS, U6.VBUS, U8.VBUS, U9.VBUS
- new net VIN_MEASURE: R45.2, R54.1, U1B.AIN7
- net +24V: now also C6.2, U$17.S, U5.IN; no longer C1.2, C47.1, D5.C, F1.2, R14.2, R15.2, R16.2, R45.1, R55.2, R56.2, R57.2, R74.2, R76.2, U$10.VIN, X12-4.S
- net +5V: now also C18.2, C19.1, U$18.VCC5V, U11.VCC, U11.~SRCLR, U1B.USB1_VBUS, U3.~EN+
- net DVI_+5V: now also U$18.5V_OUT; no longer R92.2, R93.2, RT1.2
- net ENABLE_B: now also SV2.3, U1C.GPMC_CLK; no longer SV2.4
- net ENABLE_C: now also U1C.GPMC_CSN3
- net FAN0: now also U1C.GPMC_A2
- net FAN1: now also U1C.GPMC_A3
- net FAN2: now also U1C.GPMC_AD8
- net FAN3: now also U1C.GPMC_AD9
- net FAULT_B: now also SV2.1, U1C.GPMC_A0; no longer SV2.2
- net FAULT_C: now also U1C.GPMC_AD10
- net GND: now also C14.2, C17.2, C18.1, C19.2, C5.1, C6.1, Q10.S1, Q11.S1, Q12.E, Q13.S1, Q14.S1, R142.1, R26.1, R54.2, R76.1, R91.2, R92.1, R93.1, U$18.GND, U11.GND, U11.~OE, U1B.USB1_ID, U3.GND, U4.GND, U5.COM, U5.COM_2, U5.COM_3, U5.COM_4, U6.GND, U8.GND, U9.GND, X24.DDC/CEC-GRND; no longer C102.2, C104.2, C105.1, C57.2, C58.2, C59.2, D5.A, Q1.S, Q2.S, Q3.S, Q8.S, R46.1, R47.1, R48.1, R75.1, U$11.GND, U$12.GND
- net HDMI_HPD: now also U$18.HPD_A; no longer X24.HOT_PLUG_DETECT
- net HEATER_A: now also R74.2, U1C.GPMC_OEN_REN
- net HEATER_E: now also R15.2, U1C.GPMC_ADVN_ALE
- net HEATER_H: now also R14.2, U1C.GPMC_BEN0_CLE
- net HEATER_HBP: now also R16.2, U1C.GPMC_WEN
- net N$150: no longer LED4.C, R76.1
- net N$169: now also U$18.CEC_A; no longer X24.CEC
- net N$207: now also U$18.SCL_A; no longer R92.1, X24.SCL
- net N$208: now also U$18.SDA_A; no longer R93.1, X24.SDA
- net N$234: no longer LED3.C, R55.1
- net N$242: no longer LED2.C, R56.1
- net N$64: no longer LED1.C, R57.1
- net N$8: now also Q12.C, R86.2; no longer LED8.C, R45.2
- net QUAD_ENCODER_A: now also SV5.3
- net QUAD_ENCODER_B: now also SV5.2
- net SERVO_0: now also U1C.UART0_TXD
- net SERVO_0_EN: now also U11.QE
- net SERVO_1: now also U1C.UART0_RXD
- net SERVO_1_EN: now also U11.QF
- net SPI0_CSA: no longer U$16.CSN_CFG3
- net SPI0_MISO: no longer U$13.SDO_NAO_CFG0, U$14.SDO_NAO_CFG0, U$15.SDO_NAO_CFG0, U$2.SDO_NAO_CFG0, U$9.SDO_NAO_CFG0
- net SPI0_MOSI: now also U11.SER; no longer U$13.SDI_NAI_CFG1, U$14.SDI_NAI_CFG1, U$15.SDI_NAI_CFG1, U$16.SDI_NAI_CFG1, U$9.SDI_NAI_CFG1
- net SPI0_SCLK: now also U11.SRCLK
- net SPI1_CS1: now also SV2.4; no longer SV2.3
- net SPI1_SCLK: now also SV2.2; no longer SV2.1
- net SYS_5V: no longer RT1.1, X11-1.S, X29-1.S, X7-1.S, X8-1.S
- net SYS_RESETN: no longer C105.2
- net SYS_VDD1_3V3: now also SV5.4, U$18.VCCA; no longer R1.2
- net SYS_VDD2_3V3: no longer SV5.4
- net TERM_A: now also R57.2
- net TERM_E: now also R1.2
- net TERM_H: now also R56.2
- net TERM_HBP: now also R55.2
- net TX0+: now also U$18.D0+; no longer U$12.IO4, U$12.NC5
- net TX0-: now also U$18.D0-; no longer U$12.IO3, U$12.NC4
- net TX1+: now also U$18.D1+; no longer U$11.IO2, U$11.NC2
- net TX1-: now also U$18.D1-; no longer U$11.IO1, U$11.NC1
- net TX2+: now also U$18.D2+; no longer U$11.IO4, U$11.NC5
- net TX2-: now also U$18.D2-; no longer U$11.IO3, U$11.NC4
- net TXC+: now also U$18.CLK+; no longer U$12.IO2, U$12.NC2
- net TXC-: now also U$18.CLK-; no longer U$12.IO1, U$12.NC1
- net USB1_DM3: now also U4.D+; no longer U4.IO1
- net USB1_DM4: now also U8.D+; no longer U3.IO1
- net USB1_DP: no longer R1.1
- net USB1_DP3: now also U4.D-; no longer U4.IO2
- net USB1_DP4: now also U8.D-; no longer U3.IO2
- net USB_DC: no longer C104.1
- net VDD_ADC: now also Q10.S2, Q11.S2, Q13.S2, Q14.S2; no longer R13.2, R17.2, R18.2, R77.2
- net VIN: now also D5.A, R45.1, R84.1, U$17.D; no longer F1.1, LED8.A
Other:
- note added: "Analog etc"
- note added: "To test with 25MHz clock from SIP, populate this with 0R"
- note removed: "Resettable fuse"
- moved on the sheet: C10, C100, C101, C102, C103, C108, C109, C11, C110, C111, C112, C113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

Commit message: Almost done routing. Switched to high side measurement of current
Parts:
- removed SV4: (no value), con-lstb:MA03-1
- added C20: 0.1uF, rcl:C-EUC0402
- added J2, J3: 4P-2.0, Seeed-Connector:GROVE-CONNECTOR-DIP(4P-2.0)
- added R145: 4.7K,1%, rcl:R-EU_R0402
- added R146: 47k,NTC, rcl:R-EU_R0402
- added U13: INA199A1DCKR, Texas Instruments_By_element14_Batch_1:INA199A1DCKR
- LED0, LED1, LED10, LED11, LED12, LED13, LED2, LED3, LED4, LED5, LED6, LED7, LED9: MPN Q65110A7211 -> 19-217/BHC-ZL1M2RY/3T; SPN (none) -> 19-217/BHC-ZL1M2RY/3T-ND
- R26: device resistor:R-EU_R2512 -> resistor:R-EU_R1206; MPN (none) -> ERJ-MP2MF1M0U; SPN YAG2136CT-ND -> P19339TR-ND
Connections:
- net SPI0_CSA renamed UNUSED_1
- removed net MGND: C102.2, C57.2, C58.2, C59.2, LED1.C, LED2.C, LED3.C, LED4.C, Q1.S, Q2.S, Q3.S, Q8.S, R26.2, R46.1, R47.1, R48.1, R75.1
- removed net TK_E: U1B.AIN4
- new net P-SHUNT: R26.2, U$17.S, U13.IN+
- new net THERM_BOARD: R145.2, R146.1, U1B.AIN4
- net +24V: now also R26.1, U13.IN-; no longer U$17.S
- net GND: now also C102.2, C20.1, C57.2, C58.2, C59.2, J2.4, J3.4, LED1.C, LED2.C, LED3.C, LED4.C, Q1.S, Q2.S, Q3.S, Q8.S, R114.2, R146.2, R46.1, R47.1, R48.1, R75.1, U13.GND, U13.REF; no longer R105.1, R26.1, SV4.3
- net I2C1_SCL: now also J2.1
- net I2C1_SDA: now also J2.2
- net I_MEASURE: now also U13.OUT
- net SYS_VDD1_3V3: now also C20.2, R105.1, U13.V+; no longer R114.2
- net SYS_VDD2_3V3: now also J2.3, J3.3
- net UART4_RXD: now also J3.1; no longer SV4.1
- net UART4_TXD: now also J3.2; no longer SV4.2
- net VDD_ADC: now also R145.1
Other:
- moved on the sheet: R105, R114, R26

Commit message: Working on DRC errors
Parts:
- removed H1, H2, H3, H4: MOUNT-HOLE3.2, holes:MOUNT-HOLE3.2
- removed R106, R109, R110, R111, R112, R113: 100K,1%, rcl:R-EU_R0402
- removed R24: 0R,DNI, rcl:R-EU_R0402
- removed R53: 499, OSD3358-SM-RED Platform:R-US_R0402
- added C21, C24: 0.1uF, rcl:C-EUC0402
- added C25: (no value), rcl:CPOL-EU150CLZ-0810
- added MGT1, MGT2, MGT3, MGT4: MOUNTING_HOLE, OSD3358-SM-RED Platform:MOUNTING_HOLE
- added S1: KRM_TACT_SWITCH, Manga_custom:KRM_TACT_SWITCH
- added SV1: (no value), con-lstb:MA04-1
- C100, C41, C89, C91, C92, C93: MPN C2012X5R1V106M085AC -> GMK325BJ106MN-T
- C101, C42, C94, C95, C97, C98: value 100uF -> 100uF,35V,0.025R
- C109, C111, C112, C113: MPN CL10B104KB8NNND -> GRM155R61A225KE95D
- C132: value 0.022uF -> 22nF; MPN CL10B104KB8NNND -> C1005X7R1E223K050BB
- C135: value 10uF -> 10uF,3.3V; device rcl:C-EUC0402 -> rcl:C-EUC0805; MPN CL10B104KB8NNND -> C0805C106K8PACTU
- C136: MPN CL10B104KB8NNND -> CL05B471KB5NNNC
- C138, C140, C141, C142: MPN GRM155R60J475ME47D -> CL10B104KB8NNND
- C143: value 10uF -> 10uF,3.3V; device rcl:C-EUC0402 -> rcl:C-EUC0805; MPN GRM155R60J475ME47D -> C0805C106K8PACTU
- C146, C147, C156, C157: MPN GRM155R60J475ME47D -> GRM0335C1E180JA01D
- C148, C149: MPN CL10B104KB8NNND -> GRM0335C1E180JA01D
- C22: value 0.001uF -> 4.7nF; MPN CL10B104KB8NNND -> CL05B472KA5NNNC
- C47: value 10uF -> 10uF,35V; device rcl:C-EUC1206 -> rcl:C-EUC1210; MPN CL31B106KAHNNNE -> GMK325BJ106MN-T
- IC29: MPN (none) -> LAN8710A-EZC-TR
- J2, J3: MPN (none) -> 1125S-4P
- L1: value 33uH -> 15uH; MPN NR8040T330M -> NRS8040T150MJGJ
- L2, L3: MPN (none) -> MU2029-151Y
- Q9: MPN (none) -> MMBT2907ALT3G
- R1, R140, R141, R27, R31, R35, R37, R38, R39, R40, R43, R50, R55, R56, R57, R58, R6, R60, R73, R78, R81, R88: value 10K -> 10K,1%
- R100, R101, R102, R103, R104, R85, R95, R96, R97, R98, R99: MPN RC0402JR-074K7L -> RC0402FR-07100RL
- R105, R107, R108, R114, R115, R117, R118, R119: SPN (none) -> 311-100KLRCT-ND
- R121: value 10K -> 10K,1%; MPN RC0402JR-074K7L -> RC0402FR-0710KL
- R122, R123, R124, R125: value 49.1, 1% -> 49.9,1%; MPN RC0402JR-074K7L -> RC0402FR-0749R9L
- R126, R52, R59, R70, R71, R72: MPN RC1005J2R2CS -> RC0402FR-072R2L
- R127, R128, R129, R130, R131, R132, R133, R134, R135, R136, R137, R14, R142, R15, R16, R19, R20, R21, R23, R25, R28, R32, R33, R34, R36, R44, R46, R47, R48, R5, R51, R61, R62, R63, R64, R65, R66, R67, R68, R69, R74, R75, R76, R87, R89, R92, R93: value 4.7K -> 4.7K,1%; MPN RC0402JR-074K7L -> RC0402FR-074K7L
- R13, R17, R18, R77: value 4K7, 1% -> 4.7K,1%
- R143, R144: value 4.7K -> 4.7K,1%; MPN RC1005J2R2CS -> RC0402FR-074K7L
- R145: MPN RC0402FR-0710KL -> RC0402FR-074K7L
- R146: MPN (none) -> NCP15WB473E03RC
- R149: value 0.1,5% -> 0.1R; device rcl:R-EU_R0402 -> rcl:R-EU_R0805; MPN RC1005F4422CS -> RL1220S-R10-F
- R150: MPN RC0402JR-074K7L -> RC0402JR-071ML
- R41: value 10K, 1% -> 40.2K,1%; device OSD3358-SM-RED Platform:R-US_R0402 -> rcl:R-EU_R0402; MPN (none) -> RC0402FR-0740K2L
- R49: value 40.2K, 1% -> 470; device OSD3358-SM-RED Platform:R-US_R0402 -> rcl:R-EU_R0402; MPN (none) -> RC0402JR-07470RL
- R54: value 4.7K -> 4.7K,1%; SPN 311-4.7KLRCT-ND -> (none)
- R79, R80: MPN RC0402JR-074K7L -> RC0402JR-07470RL
- R82: MPN RC0402FR-0710KL -> RC0402FR-0712K1L
- R83: value 10 -> 10,1%; MPN RC0402JR-074K7L -> RC0402FR-0710RL
- R91: value 4.7K -> 4.7K,1%; MPN (none) -> RC0402FR-074K7L
- S3, S4: MPN (none) -> KMR241G ULC LFS
- SV2, SV3: value (none) -> DNI
- U$10: MPN (none) -> TPS54202DDCR
- U$13, U$14, U$15, U$16, U$9: MPN (none) -> TMC2130-LA-T; SPN 1460-1130-2-ND -> (none)
- U$17: MPN (none) -> SISS27DN-T1-GE3
- U$18: MPN (none) -> TPD12S016RKTR
- U$2: MPN TMC2130-LA -> TMC2130-LA-T; SPN 1460-1130-2-ND -> (none)
- U$3: MPN (none) -> LPJ0011BBNL
- U$5, U$6: MPN (none) -> 0672983090
- U$7: MPN (none) -> TDA19988BHN/C1,518
- U$8: MPN (none) -> 10118193-0001LF
- U1: MPD OSD3358-512M-BAS000 -> (none); MPN (none) -> OSD3358-512M-BSM
- U10: value TPD4S012_DRY_6 -> TPD4S012_DRY_6_P1_P; device BeagleBone_Blue:TPD4S012_DRY_6 -> OSD3358-SM-RED Platform:TPD4S012_DRY_6_P1_P; MPN (none) -> TPD4S012DRYR
- U4, U6, U8, U9: MPN (none) -> TPD4S012DRYR
- U7: MPN (none) -> TLVH431IDBZR
- VDDS_PLL, VDD_MPU: value TPB1,27 -> TPTP06R; device testpad:TPB1,27 -> testpad:TPTP06R
- Y1, Y2: MPN (none) -> 445C33D25M00000
- Y4: MPN (none) -> NX8045GB-6MHZ-STD-CSF-3
- renumbered C152 to C22
Connections:
- removed net FAULT_B: SV2.1, U1C.GPMC_A0
- removed net FAULT_C: SV3.1, U1C.GPMC_AD10
- removed net PMIC_SCL: U1A.I2C0_SCL, U1A.PMIC_SCL
- removed net PMIC_SDA: U1A.I2C0_SDA, U1A.PMIC_SDA
- removed net TK_H: U1B.AIN5
- removed net TRSRTN: J1.TRSTN
- removed net UNUSED_1: U1D.RMII1_REF_CLK
- removed net USB1_DRVVBUS: U1B.USB1_DRVVBUS
- removed net USB_RESET: R88.1, U2.~RESET
- removed net VDD_3V3B: R90.1
- new net PMIC_MUX: U1B.AIN5, U1B.PMIC_MUX_IN
- net +5V: no longer C18.2, C19.1, C82.1, C83.1, IC6P.VCC, IC7P.VCC, R61.2, R62.2, R63.2, R64.2, R65.2, R66.2, U$18.VCC5V, U11.VCC, U11.~SRCLR, U3.~EN+, X1-3.S, X10-3.S, X12-3.S, X13-3.S, X19-3.S, X22-3.S
- net CGND: now also MGT1.P$1, MGT2.P$1, MGT3.P$1, MGT4.P$1
- net CLKOUT2_48MHZ: no longer U2.TSTPLL/48MCLK
- net DVI_+5V: now also C21.1
- net ENABLE_B: now also U11.QG; no longer U1C.GPMC_CLK
- net ENABLE_C: now also U11.QH; no longer U1C.GPMC_CSN3
- net FAULT_A: now also U1C.GPMC_AD10
- net FAULT_E: now also U1C.GPMC_CLK
- net FAULT_H: now also U1D.RMII1_REF_CLK
- net FAULT_Y: now also U1C.GPMC_CSN3
- net FAULT_Z: now also U1C.GPMC_A0
- net GND: now also C21.2, C24.2, C25.-, R117.2, S1.2, SV1.1, SV2.1, SV3.1; no longer R106.1, R109.1, R110.1, R111.1, R112.1, R113.1, U10.GND
- net HDMI_HPD: now also U$18.LS_OE
- net I2C0_SCL: now also U1A.I2C0_SCL, U1A.PMIC_SCL
- net I2C0_SDA: now also U1A.I2C0_SDA, U1A.PMIC_SDA
- net LCD_D10: no longer R110.2
- net LCD_D11: no longer R109.2
- net LCD_D2: now also S1.1
- net LCD_D6: no longer R106.2
- net LCD_D7: no longer R113.2
- net LCD_D8: no longer R112.2
- net LCD_D9: no longer R111.2
- net N$1: now also R88.2; no longer R49.2
- net N$192: no longer R24.2
- net N$4: now also R49.2; no longer R53.1
- net SERVO_0: now also SV1.3
- net SERVO_1: now also SV1.4
- net SYS_5V: now also C18.2, C19.1, C24.1, C25.+, C82.1, C83.1, IC6P.VCC, IC7P.VCC, R61.2, R62.2, R63.2, R64.2, R65.2, R66.2, U$18.VCC5V, U11.VCC, U11.~SRCLR, U3.~EN+, X1-3.S, X10-3.S, X12-3.S, X13-3.S, X19-3.S, X22-3.S
- net SYS_RESETN: now also U2.~RESET
- net SYS_RTC_1V8: now also R41.2; no longer R49.1
- net SYS_VDD1_3V3: now also R90.1, U$18.CT_HPD; no longer R117.2, R24.1, R88.2, SV5.4
- net SYS_VDD2_3V3: now also SV1.2, SV5.4
- net SYS_VDD3_3V3: now also R49.1, R88.1; no longer R41.2, R53.2
- net TRSTN: now also J1.TRSTN
- net USB0_DM: now also U10.D+; no longer U10.D-
- net USB0_DP: now also U10.D-; no longer U10.D+
Other:
- moved on the sheet: C1, C135, C143, R115, R116, R117, R118, R119, R120, R144, R88, R90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
