File: PCB/Revolve_A0/Revolve_A0.sch (EAGLE design)
At the start: 382 parts, among them IC29 LAN8710A, IC30 MTFC2GMDEA, IC6 74AHC1G126DCK, IC7 74AHC1G126DCK, J2 4P-2.0, J3 4P-2.0, Q1 AON6758, Q10 DMC2038LVT, Q11 DMC2038LVT, Q13 DMC2038LVT, Q14 DMC2038LVT, Q2 AON6758, Q3 AON6758, Q8 AON6758, Q9 MMBT2907, U1 OSD3358-512M-BSM, U10 TPD4S012_DRY_6_P1_P, U11 SN74AHC595PW, U13 INA199A1DCKR, U19 CD4050BD, U2 TUSB2046BIRHBT, U3 TPS2061D, U4 TPD4S012_DRY_6_P1_P, U5 UA78L05ACD, U6 TPD4S012_DRY_6_P1_P, U7 TLVH431, U8 TPD4S012_DRY_6_P1_P, U9 TPD4S012_DRY_6_P1_P, X1 22-05-7038-03, X10 22-05-7038-03, X11 22-05-7038-03, X12 22-05-7048-04, X13 22-05-7038-03, X14 22-05-7048-04, X15 22-05-7048-04, X16 22-05-7048-04, X17 22-05-7048-04, X18 22-05-7048-04, X19 22-05-7038-03, X2 MSTBA4, X20 MSTBA4, X21 MSTBA2, X22 22-05-7038-03, X24 HDMI4, X25 22-05-7048-04, X26 MSTBA2, X29 22-05-7038-03, X3 MSTBA2, X4 22-05-7028-02, X5 22-05-7028-02, X6 22-05-7028-02, X7 22-05-7038-03, X8 22-05-7038-03, X9 22-05-7028-02, Y1 25MHz, Y2 25MHz, Y4 6 MHz

Commit message: REady for board review
Parts:
- added C27: 0.1uF, rcl:C-EUC0402
- PMIC_NRESET, SYS_5V, SYS_VDD1_3V3, VDDS_DDR, VDD_CODE: value TPB1,27 -> TPTP06R; device testpad:TPB1,27 -> testpad:TPTP06R
Connections:
- net GND: now also C27.2
- net SYS_VDD1_3V3: now also C27.1
Changed lines of the file:
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@@
 <part name="P+8" library="supply1" deviceset="+24V" device=""/>
 <part name="P+9" library="supply1" deviceset="+24V" device=""/>
-<part name="P+10" library="supply1" deviceset="+5V" device=""/>
-<part name="P+11" library="supply1" deviceset="+5V" device=""/>
 <part name="P+12" library="supply1" deviceset="+5V" device=""/>
-<part name="P+13" library="supply1" deviceset="+5V" device=""/>
 <part name="+3V29" library="supply1" deviceset="+3V3" device=""/>
 <part name="C107" library="rcl" deviceset="C-EU" device="C0402" value="0.1uF">
@@
 <attribute name="MPN" value="NX8045GB-6MHZ-STD-CSF-3"/>
 </part>
-<part name="P+16" library="supply1" deviceset="+5V" device=""/>
-<part name="P+18" library="supply1" deviceset="+5V" device=""/>
 <part name="L2" library="rcl" deviceset="L-US" device="L2012C" value="150OHM,800mA">
 <attribute name="MPN" value="MU2029-151Y"/>
@@
 <attribute name="MPN" value="RL1220S-R10-F"/>
 </part>
-<part name="SYS_5V" library="testpad" deviceset="TP" device="B1,27" value="TPB1,27"/>
-<part name="SYS_VDD1_3V3" library="testpad" deviceset="TP" device="B1,27" value="TPB1,27"/>
+<part name="SYS_5V" library="testpad" deviceset="TP" device="TP06R" value="TPTP06R"/>
+<part name="SYS_VDD1_3V3" library="testpad" deviceset="TP" device="TP06R" value="TPTP06R"/>
 <part name="SYS_VDD2_3V3" library="testpad" deviceset="TP" device="B1,27" value="TPB1,27"/>
 <part name="SYS_VDD3_3V3" library="testpad" deviceset="TP" device="B1,27" value="TPB1,27"/>
@@
 </part>
 <part name="EEPROM_WP" library="testpad" deviceset="TP" device="B1,27" value="TPB1,27"/>
-<part name="VDDS_DDR" library="testpad" deviceset="TP" device="B1,27" value="TPB1,27"/>
-<part name="VDD_CODE" library="testpad" deviceset="TP" device="B1,27" value="TPB1,27"/>
+<part name="VDDS_DDR" library="testpad" deviceset="TP" device="TP06R" value="TPTP06R"/>
+<part name="VDD_CODE" library="testpad" deviceset="TP" device="TP06R" value="TPTP06R"/>
 <part name="VDD_MPU" library="testpad" deviceset="TP" device="TP06R" value="TPTP06R"/>
 <part name="VDDS_PLL" library="testpad" deviceset="TP" device="TP06R" value="TPTP06R"/>
-<part name="PMIC_NRESET" library="testpad" deviceset="TP" device="B1,27" value="TPB1,27"/>
+<part name="PMIC_NRESET" library="testpad" deviceset="TP" device="TP06R" value="TPTP06R"/>
 <part name="GND37" library="supply1" deviceset="GND" device=""/>
 <part name="U$8" library="Manga_screen_rev_B-3" deviceset="USB-MICRO" device="">
@@
 <attribute name="MPN" value="KMR241G ULC LFS"/>
 </part>
+<part name="C27" library="rcl" deviceset="C-EU" device="C0402" value="0.1uF">
+<attribute name="MPN" value="CL10B104KB8NNND"/>
+</part>
+<part name="GND174" library="supply1" deviceset="GND" device=""/>
 </parts>
 <sheets>
@@
 <instance part="P+8" gate="1" x="1000.76" y="360.68"/>
 <instance part="P+9" gate="1" x="1069.34" y="358.14"/>
-<instance part="P+10" gate="1" x="947.42" y="741.68"/>
-<instance part="P+11" gate="1" x="1018.54" y="767.08"/>
 <instance part="P+12" gate="1" x="551.18" y="160.02"/>
-<instance part="P+13" gate="1" x="1145.54" y="769.62"/>
 <instance part="+3V29" gate="G$1" x="490.22" y="396.24"/>
 <instance part="C107" gate="G$1" x="541.02" y="685.8" smashed="yes">
@@
 <attribute name="MPN" x="502.92" y="993.14" size="1.778" layer="96" display="off"/>
 </instance>
-<instance part="P+16" gate="1" x="1023.62" y="220.98"/>
-<instance part="P+18" gate="1" x="1104.9" y="736.6"/>
 <instance part="L2" gate="G$1" x="927.1" y="1005.84" rot="R90">
 <attribute name="MPN" x="927.1" y="1005.84" size="1.778" layer="96" rot="R90" display="off"/>
@@
 <attribute name="MPN" x="525.78" y="309.88" size="1.778" layer="96" display="off"/>
 </instance>
+<instance part="C27" gate="G$1" x="276.86" y="944.88" rot="MR0">
+<attribute name="MPN" x="276.86" y="944.88" size="1.778" layer="96" rot="MR0" display="off"/>
+</instance>
+<instance part="GND174" gate="1" x="276.86" y="937.26"/>
 </instances>
 <busses>
@@
 <pinref part="GND173" gate="1" pin="GND"/>
 </segment>
+<segment>
+<pinref part="C27" gate="G$1" pin="2"/>
+<pinref part="GND174" gate="1" pin="GND"/>
+</segment>
 </net>
 <net name="N$114" class="0">
@@
 <pinref part="X13" gate="-3" pin="S"/>
 <wire x1="970.28" y1="718.82" x2="993.14" y2="718.82" width="0.1524" layer="91"/>
-<pinref part="P+10" gate="1" pin="+5V"/>
+<label x="947.42" y="739.14" size="1.778" layer="95" xref="yes"/>
 </segment>
 <segment>
@@
 <wire x1="1018.54" y1="759.46" x2="1018.54" y2="764.54" width="0.1524" layer="91"/>
 <junction x="1018.54" y="759.46"/>
-<pinref part="P+11" gate="1" pin="+5V"/>
+<label x="1018.54" y="764.54" size="1.778" layer="95" xref="yes"/>
 </segment>
 <segment>
@@
 <wire x1="1137.92" y1="762" x2="1145.54" y2="762" width="0.1524" layer="91"/>
 <junction x="1145.54" y="762"/>
-<pinref part="P+13" gate="1" pin="+5V"/>
+<label x="1145.54" y="767.08" size="1.778" layer="95" xref="yes"/>
 </segment>
 <segment>
@@
 <pinref part="X12" gate="-3" pin="S"/>
 <wire x1="1127.76" y1="718.82" x2="1153.16" y2="718.82" width="0.1524" layer="91"/>
-<pinref part="P+18" gate="1" pin="+5V"/>
+<label x="1104.9" y="734.06" size="1.778" layer="95" xref="yes"/>
 </segment>
 <segment>
@@
 <wire x1="1023.62" y1="213.36" x2="1023.62" y2="218.44" width="0.1524" layer="91"/>
 <junction x="1023.62" y="213.36"/>
-<pinref part="P+16" gate="1" pin="+5V"/>
+<label x="1023.62" y="218.44" size="1.778" layer="95" xref="yes"/>
 </segment>
 <segment>
@@
 <wire x1="276.86" y1="947.42" x2="284.48" y2="947.42" width="0.1524" layer="91"/>
 <junction x="284.48" y="947.42"/>
+<pinref part="C27" gate="G$1" pin="1"/>
+<junction x="276.86" y="947.42"/>
 </segment>
 <segment>

Commit message: Added readme
Connections:
- net CLKOUT2_48MHZ renamed UNUSED_1
Changed lines of the file:
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@@
 </segment>
 </net>
-<net name="CLKOUT2_48MHZ" class="0">
+<net name="UNUSED_1" class="0">
 <segment>
 <pinref part="U1" gate="C" pin="XDMA_EVENT_INTR1"/>

Commit message: Ordered PCB and stencil + parts from OSH park/Digi key
Parts:
- removed Q12: (no value), semicon-smd-ipc:NPN-TRANSISTOR_SOT23
- added R106, R109, R110, R111, R153, R154, R155, R53: 1K,1%, rcl:R-EU_R0402
- added R24: 4.7K,1%, rcl:R-EU_R0402
- added T1: (no value), zetex:NMOSSOT23
- added U$11: SISS27DN, Revolve:SISS27DN
- C1, C10, C107, C108, C110, C114, C115, C12, C13, C133, C134, C138, C140, C141, C142, C15, C150, C151, C155, C16, C18, C19, C2, C20, C21, C23, C24, C27, C28, C30, C35, C38, C4, C40, C44, C5, C53, C54, C56, C6, C60, C61, C63, C64, C66, C67, C69, C70, C72, C73, C74, C8, C82, C83, C84, C85, C87, C99: PARTNO (none) -> GRM155R71H103KA88J
- C100, C41, C89, C91, C92, C93: PARTNO (none) -> C0805C106K8PACTU
- C137: MPN CL10B104KB8NNND -> CL05A105MP5NNNC
- C32: PARTNO (none) -> GRM155R71H103KA88J; VID (none) -> 490-6351-2-ND
- R2: PARTNO (none) -> *
- R84: SPN 311-100KLRCT-ND -> (none)
- R86: value 100K,1% -> 40.2K,1%; MPN RC0402FR-07100KL -> RC0402FR-0740K2L; SPN 311-100KLRCT-ND -> (none)
- U$18: MPN TPD12S016RKTR -> TPD12S016PWR
- X24: PARTNO (none) -> 10029449-111RLF
Connections:
- removed net N$212: IC29.RXD3/PHYAD2, R95.1
- removed net N$225: IC29.RXD2/RMIISEL, R96.1
- removed net N$226: IC29.RXD1/MODE1, R97.1
- removed net N$227: IC29.RXD0/MODE0, R99.1
- removed net N$229: IC29.RXCLK/PHYAD1, R100.1
- removed net N$230: IC29.RXER/RXD4/PHYAD0, R101.1
- removed net N$239: IC29.COL/CRS_DV/MODE2, R103.1
- new net MODE2: IC29.COL/CRS_DV/MODE2, R103.1, R155.2
- new net N$17: R24.2, R53.1, U$17.G
- new net REFCLK0: IC29.RXCLK/PHYAD1, R100.1, R106.2
- new net RXD0: IC29.RXD0/MODE0, R153.2, R99.1
- new net RXD1: IC29.RXD1/MODE1, R154.2, R97.1
- new net RXD2: IC29.RXD2/RMIISEL, R109.2, R96.1
- new net RXD3: IC29.RXD3/PHYAD2, R110.2, R95.1
- new net RXER: IC29.RXER/RXD4/PHYAD0, R101.1, R111.2
- new net VMID: R24.1, R84.1, U$11.S, U$17.S
- net ENABLE_STUFF: now also T1.G; no longer Q12.B
- net GND: now also R106.1, R109.1, R110.1, R111.1, R53.2, T1.S; no longer Q12.E
- net N$26: now also U$11.G; no longer U$17.G
- net N$8: now also T1.D; no longer Q12.C
- net P-SHUNT: now also U$11.D; no longer U$17.S
- net SYS_5V: now also U3.IN, U3.IN_2; no longer U3.~EN+
- net SYS_VDD1_3V3: now also R153.1, R154.1, R155.1
- net USB_PWR: now also U3.~EN+; no longer U3.IN, U3.IN_2
- net VIN: no longer R84.1
Other:
- note added: "Configuration"
- note added: "IO_VOLT_SEL"
- note added: "MODE[0]"
- note added: "MODE[1]"
- note added: "MODE[2]"
- note added: "MODE[3]"
- note added: "PHY_ADDR0"
- note added: "PHY_ADDR1"
- note added: "PHY_ADDR2"
- moved on the sheet: C18, R100, R101, R102, R103, R104, R45, R54, R91, R95, R96, R97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
