File: PCB/Revolve_A5/Revolve_A5.sch (KiCad schematic (older format))
At the start: 413 parts, among them IC1 741G126DCK, IC2 CY7C65632, IC29 LAN8710A, IC30 MTFC2GMDEA, IC6 741G126DCK, IC7 741G126DCK, J1 CTI-JTAG, J2 4P-2.0, J3 4P-2.0, Q1 AON6758, Q10 DMC2038LVT, Q11 DMC2038LVT, Q12 AON6792, Q13 DMC2038LVT, Q14 DMC2038LVT, Q15 AON6792, Q16 DMC2038LVT, Q2 AON6758, Q3 AON6758, Q4 NPN-TRANSISTOR_SOT23, Q5 NPN-TRANSISTOR_SOT23, Q6 NPN-TRANSISTOR_SOT23, Q7 NPN-TRANSISTOR_SOT23, Q8 AON6758, Q9 MMBT2907, U1 OSD3358-512M-BSM, U10 TPD4S012_DRY_6_P1_P, U11 SN74AHC595PW, U12 APX811SOT, U13 INA199A1DCKR, U19 CD4050BD, U2 TCK401G,LF, U3 TPS2061D, U4 TPD4S012_DRY_6_P1_P, U5 UA78L05ACD, U6 TPD4S012_DRY_6_P1_P, U7 TLVH431, U8 TPD4S012_DRY_6_P1_P, U9 TPD4S012_DRY_6_P1_P, X1 22-?-0305-7038, X10 22-?-0305-7038, X11 22-?-0305-7038, X12 22-?-0405-7048, X13 22-?-0305-7038, X14 22-?-0405-7048, X15 22-?-0405-7048, X16 22-?-0405-7048, X17 22-?-0405-7048, X18 22-?-0405-7048, X19 22-?-0305-7038, X2 MSTBA4, X20 MSTBA4, X21 MSTBA2, X22 22-?-0305-7038, X24 HDMI4, X25 22-?-0405-7048, X26 MSTBA2, X29 22-?-0305-7038, X3 MSTBA2, X4 22-?-0205-7028, X5 22-?-0205-7028, X6 22-?-0205-7028, X7 22-?-0305-7038, X8 22-?-0305-7038, X9 22-?-0205-7028, Y1 25MHz, Y2 25MHz

Commit message: Added files needed for Umikaze.
Parts:
- Q12, Q15: SPN (none) -> 785-1744-1-ND
- R26: SPN (none) -> 696-1369-1-ND
- U2: SPN (none) -> TCK401GLFCT-ND
